File: umiko.sch (KiCad schematic (older format))
At the start: 366 parts, among them J1 MJ-4PP-9, J2 MJ-4PP-9, U1 proton_c, U2 proton_c

Commit message: more wiring
Parts:
- LED1, LED10, LED100, LED101, LED102, LED103, LED104, LED11, LED12, LED13, LED14, LED15, LED16, LED17, LED18, LED19, LED2, LED20, LED21, LED22, LED23, LED24, LED25, LED26, LED27, LED28, LED29, LED3, LED30, LED31, LED32, LED33, LED34, LED35, LED36, LED37, LED38, LED39, LED4, LED40, LED41, LED42, LED43, LED44, LED45, LED46, LED47, LED48, LED49, LED5, LED50, LED51, LED52, LED53, LED54, LED55, LED56, LED57, LED58, LED59, LED6, LED60, LED61, LED62, LED63, LED64, LED65, LED66, LED67, LED68, LED69, LED7, LED70, LED71, LED72, LED73, LED74, LED75, LED76, LED77, LED78, LED79, LED8, LED80, LED81, LED82, LED83, LED84, LED85, LED86, LED87, LED88, LED89, LED9, LED90, LED91, LED92, LED93, LED94, LED95, LED96, LED97, LED98, LED99: symbol bakekujira-rescue:YS-SK6812MINI-E-kbd -> umiko-rescue:YS-SK6812MINI-E-kbd
- OL1, OL2: symbol bakekujira-rescue:OLED-kbd -> umiko-rescue:OLED-kbd
- RSW1, RSW2: symbol bakekujira-rescue:SW_PUSH-kbd -> umiko-rescue:SW_PUSH-kbd
- SW_1, SW_10, SW_11, SW_12, SW_13, SW_14, SW_15, SW_16, SW_17, SW_18, SW_19, SW_2, SW_20, SW_21, SW_22, SW_23, SW_24, SW_26, SW_27, SW_28, SW_3, SW_30, SW_31, SW_32, SW_33, SW_34, SW_35, SW_36, SW_37, SW_38, SW_39, SW_4, SW_40, SW_43, SW_44, SW_45, SW_46, SW_47, SW_48, SW_49, SW_5, SW_50, SW_51, SW_52, SW_54, SW_56, SW_57, SW_58, SW_59, SW_6, SW_60, SW_66, SW_67, SW_68, SW_8, SW_9: footprint kbd:CherryMX_Hotswap -> onigaku:CherryMX_Hotswap
- SW_25, SW_29: footprint kbd:CherryMX_Hotswap_1.5u -> onigaku:CherryMX_Hotswap_1.5u
- SW_41, SW_55: footprint kbd:CherryMX_Hotswap_2.25u_North -> onigaku:CherryMX_Hotswap_2.25u_North
- SW_42: footprint kbd:CherryMX_Hotswap_1.75u -> onigaku:CherryMX_Hotswap_1.75u
- SW_53: footprint kbd:CherryMX_Hotswap_2.75u_North -> onigaku:CherryMX_Hotswap_2.75u_North
- SW_61: footprint kbd:CherryMX_Hotswap_2.75u_North_reversed_stabilizers -> onigaku:CherryMX_Hotswap_2.75u_North_reversed_stabilizers
- SW_62, SW_63, SW_64, SW_65, SW_69, SW_70, SW_71, SW_72: footprint kbd:CherryMX_Hotswap_1.25u_North -> onigaku:CherryMX_Hotswap_1.25u_North
- SW_7: footprint kbd:CherryMX_Hotswap_2u_North -> onigaku:CherryMX_Hotswap_2u_North
- SW_73: footprint kbd:CherryMX_Hotswap_2.25u_North_reversed_stabilizers -> onigaku:CherryMX_Hotswap_2.25u_North_reversed_stabilizers
