File: umiko.kicad_pcb (KiCad board)
At the start: 2 copper layers, 405.8 x 120.8 mm, 366 parts, among them J1 MJ-4PP-9, J2 MJ-4PP-9, U1 proton_c, U2 proton_c

Commit message: 4 layers, incorporating design
Parts:
- removed D_10, D_26, D_27, D_28, D_54, D_66, D_67, D_68, D_8, D_9: D, kbd:D3_SMD_v2
- removed LED21, LED24, LED25, LED5, LED6: YS-SK6812MINI-E, kbd:YS-SK6812MINI-E_underglow
- removed LED38, LED39, LED40, LED56, LED57, LED58, LED85, LED96, LED97, LED98: YS-SK6812MINI-E, kbd:YS-SK6812MINI-E
- removed RSW2: SW_PUSH, Button_Switch_SMD:SW_SPST_TL3342
- removed SW_10, SW_26, SW_27, SW_28, SW_54, SW_66, SW_67, SW_68, SW_8, SW_9: KEYSW, onigaku:CherryMX_Hotswap
- added C105: 100n, Capacitor_SMD:C_0402_1005Metric, F.Cu at (173.8, 70.3)
- added C106: 100n, Capacitor_SMD:C_0402_1005Metric, F.Cu at (171.3, 80.3)
- added C3: 0.1uF, Capacitor_SMD:C_0603_1608Metric_Pad1.08x0.95mm_HandSolder, F.Cu at (196.8, 0.31)
- added C4: 0.1uF, Capacitor_SMD:C_0603_1608Metric_Pad1.08x0.95mm_HandSolder, F.Cu at (196.8, 2.82)
- added C5b1: 10u, Capacitor_SMD:C_0402_1005Metric, F.Cu at (172.9, 63.6)
- added C6_A1: 100n, Capacitor_SMD:C_0402_1005Metric, F.Cu at (174.9, 64.9)
- added C6b1: 4.7u, Capacitor_SMD:C_0402_1005Metric, F.Cu at (164.6, 60.7)
- added D1: Power LED, Diode_SMD:D_0402_1005Metric, F.Cu at (175.8, 70.4)
- added D2: User LED, Diode_SMD:D_0402_1005Metric, F.Cu at (174.9, 70.3)
- added D3: PMEG2010BELD, PCM_0xcb:SOD882D, B.Cu at (59.6, 37.7)
- added F1: 500mA, Fuse:Fuse_0603_1608Metric, B.Cu at (58.8, 38.8)
- added FB1: 600R, Resistor_SMD:R_0402_1005Metric, F.Cu at (184.3, 16.8)
- added J4: USB_C_Receptacle_USB2.0_16P_TRRS, PCM_marbastlib-various:USB_C_Receptacle_HRO_TYPE-C-31-M-12, F.Cu at (364.7, 60.5)
- added J5: USB_C_Receptacle_USB2.0, PCM_0xcb:USB_C_Receptacle_HRO_TYPE-C-31-M-12, F.Cu at (54.4, 32.0)
- added JP1: SolderJumper_2_Open, Jumper:SolderJumper-2_P1.3mm_Open_TrianglePad1.0x1.5mm, F.Cu at (164.4, 65.3)
- added LED3: YS-SK6812MINI-E, onigaku:YS-SK6812MINI-E_underglow, F.Cu at (186.2, 7.83)
- added LED4: YS-SK6812MINI-E, onigaku:YS-SK6812MINI-E_underglow, F.Cu at (186.2, 12.6)
- added Q1: 2N7002VC-, PCM_0xcb:SOT-563, F.Cu at (172.9, 80.7)
- added Q2: 2N7002VC-, PCM_0xcb:SOT-563, F.Cu at (166.7, 62.5)
- added R10: 1k, Resistor_SMD:R_0402_1005Metric, F.Cu at (175.8, 68.5)
- added R11: 10k, Resistor_SMD:R_0402_1005Metric, F.Cu at (166.3, 65.6)
- added R12: 27, Resistor_SMD:R_0402_1005Metric, F.Cu at (168.8, 63.1)
- added R13: 27, Resistor_SMD:R_0402_1005Metric, F.Cu at (171.6, 63.1)
- added R14: 1k, Resistor_SMD:R_0402_1005Metric, F.Cu at (168.8, 80.0)
- added R15: 1k, Resistor_SMD:R_0402_1005Metric, F.Cu at (174.9, 68.5)
- added R16: 5.1k, Resistor_SMD:R_0402_1005Metric, F.Cu at (175.1, 77.6)
- added R17: 10k, Resistor_SMD:R_0402_1005Metric, F.Cu at (175.1, 78.5)
- added R3_L1: 10k, Resistor_SMD:R_0402_1005Metric, F.Cu at (171.3, 82.2)
- added R3b1: 10k, Resistor_SMD:R_0402_1005Metric, F.Cu at (172.9, 82.5)
- added R4_L1: 51k, Resistor_SMD:R_0402_1005Metric, F.Cu at (165.1, 63.0)
- added R4b1: 10k, Resistor_SMD:R_0402_1005Metric, F.Cu at (167.9, 63.1)
- added R5: 51k, Resistor_SMD:R_0402_1005Metric, F.Cu at (164.6, 61.6)
- added R6: 51k, Resistor_SMD:R_0402_1005Metric, F.Cu at (164.1, 63.0)
- added R7: 5.1k, Resistor_SMD:R_0402_1005Metric, F.Cu at (181.0, 2.06)
- added R8: 5.1k, Resistor_SMD:R_0402_1005Metric, F.Cu at (181.0, 4.05)
- added R9: 1k, Resistor_SMD:R_0402_1005Metric, F.Cu at (166.5, 64.2)
- added SW1: SWITCH, PCM_0xcb:1.9x2.8mm SW, F.Cu at (175.0, 81.0)
- added TP1: CLK, PCM_0xcb:TestPoint_Pad_D0.8mm, F.Cu at (196.0, 7.96)
- added TP2: DIO, PCM_0xcb:TestPoint_Pad_D0.8mm, F.Cu at (196.0, 10.7)
- added U3: W25Q128JVPIQ, PCM_0xcb:W25Q128JVPIQ, F.Cu at (170.4, 66.9)
- added U4: RP2040, Package_DFN_QFN:QFN-56-1EP_7x7mm_P0.4mm_EP3.2x3.2mm, F.Cu at (170.1, 75.2)
- added U5: 74LVC1T45, PCM_0xcb:SOT-563, F.Cu at (165.4, 68.3)
- added Y1: 12MHz, Crystal:Crystal_SMD_2520-4Pin_2.5x2.0mm, F.Cu at (168.0, 81.8)
- C21, R3: moved to F.Cu
- C26, C29: value 0.1uF -> 10u; footprint Capacitor_SMD:C_0603_1608Metric_Pad1.08x0.95mm_HandSolder -> Capacitor_SMD:C_0402_1005Metric; moved to F.Cu
- C30, C38: value 0.1uF -> 15p; footprint Capacitor_SMD:C_0603_1608Metric_Pad1.08x0.95mm_HandSolder -> Capacitor_SMD:C_0402_1005Metric; moved to F.Cu
- C39, C40: value 0.1uF -> 1u; footprint Capacitor_SMD:C_0603_1608Metric_Pad1.08x0.95mm_HandSolder -> Capacitor_SMD:C_0402_1005Metric; moved to F.Cu
- C5: value 0.1uF -> 10u; footprint Capacitor_SMD:C_0603_1608Metric_Pad1.08x0.95mm_HandSolder -> Capacitor_SMD:C_0402_1005Metric
- C56, C57, C58, C85, C96, C97, C98: value 0.1uF -> 100n; footprint Capacitor_SMD:C_0603_1608Metric_Pad1.08x0.95mm_HandSolder -> Capacitor_SMD:C_0402_1005Metric; moved to F.Cu
- D_1, D_11, D_12, D_13, D_14, D_15, D_16, D_17, D_18, D_19, D_2, D_20, D_21, D_22, D_23, D_24, D_25, D_29, D_3, D_30, D_31, D_32, D_33, D_34, D_35, D_36, D_37, D_38, D_39, D_4, D_40, D_41, D_42, D_43, D_44, D_45, D_46, D_47, D_48, D_49, D_5, D_50, D_51, D_52, D_53, D_55, D_56, D_57, D_58, D_59, D_6, D_60, D_61, D_62, D_63, D_64, D_65, D_69, D_7, D_70, D_71, D_72, D_73: footprint kbd:D3_SMD_v2 -> onigaku:D3_SMD_v2
- J2: moved to B.Cu
- LED1, LED10, LED104, LED11, LED12, LED13, LED14, LED15, LED16, LED17, LED18, LED19, LED2, LED20, LED22, LED23, LED26, LED27, LED28, LED29, LED30, LED7, LED8, LED9: footprint kbd:YS-SK6812MINI-E_underglow -> onigaku:YS-SK6812MINI-E_underglow
- LED100, LED101, LED102, LED103, LED31, LED32, LED33, LED34, LED35, LED36, LED37, LED41, LED42, LED43, LED44, LED45, LED46, LED47, LED48, LED49, LED50, LED51, LED52, LED53, LED54, LED55, LED59, LED60, LED61, LED62, LED63, LED64, LED65, LED66, LED67, LED68, LED69, LED70, LED71, LED72, LED73, LED74, LED75, LED76, LED77, LED78, LED79, LED80, LED81, LED82, LED83, LED84, LED86, LED87, LED88, LED89, LED90, LED91, LED92, LED93, LED94, LED95, LED99: footprint kbd:YS-SK6812MINI-E -> onigaku:YS-SK6812MINI-E
- OL1, OL2: footprint kbd:OLED_v2 -> onigaku:OLED_v2
- U1: value proton_c -> USBLC6-2P6; footprint proton_c:proton_c -> Package_TO_SOT_SMD:SOT-666; moved to F.Cu
- U2: value proton_c -> TLV75533PDQNR; footprint proton_c:proton_c -> PCM_0xcb:X2SON-4; moved to F.Cu
- moved C5 294.0 mm to (57.8, 37.7), turned to 0 degrees
- moved U1 246.6 mm to (170.3, 63.0), turned to 90 degrees
- moved C98 236.5 mm to (169.6, 70.3)
- moved C40 231.7 mm to (171.7, 70.3), turned to -90 degrees
- moved C30 227.8 mm to (170.4, 82.1)
- moved C58 226.7 mm to (175.1, 72.7), turned to 0 degrees
- moved C29 224.0 mm to (175.4, 63.5), turned to -90 degrees
- moved C97 220.7 mm to (166.8, 70.2)
- moved C85 213.8 mm to (170.5, 70.3)
- moved C39 211.8 mm to (172.7, 70.3), turned to -90 degrees
- moved C57 208.1 mm to (175.1, 76.3), turned to 0 degrees
- moved C96 202.6 mm to (165.1, 76.2), turned to 180 degrees
- moved C38 201.8 mm to (165.9, 82.3), turned to -90 degrees
- moved C26 194.4 mm to (166.5, 60.7), turned to 0 degrees
- moved C56 194.0 mm to (170.4, 80.3), turned to -90 degrees
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Connections:
- C1 pad 1: VDD -> 5V_R
- C1 pad 2: GNDA -> GND_R
- C10 pad 1: GND -> GND_L
- C10 pad 2: VCC -> 5V_L
- C100 pad 1: VCC -> 5V_L
- C100 pad 2: GND -> GND_L
- C101 pad 1: VCC -> 5V_L
- C101 pad 2: GND -> GND_L
- C102 pad 1: VCC -> 5V_L
- C102 pad 2: GND -> GND_L
- C103 pad 1: VCC -> 5V_L
- C103 pad 2: GND -> GND_L
- C104 pad 1: VDD -> 5V_R
- C104 pad 2: GNDA -> GND_R
- C11 pad 1: GND -> GND_L
- C11 pad 2: VCC -> 5V_L
- C12 pad 1: VCC -> 5V_L
- C12 pad 2: GND -> GND_L
- C13 pad 1: GND -> GND_L
- C13 pad 2: VCC -> 5V_L
- C14 pad 1: VDD -> 5V_R
- C14 pad 2: GNDA -> GND_R
- C15 pad 1: GND -> GND_L
- C15 pad 2: VCC -> 5V_L
- C16 pad 1: GND -> GND_L
- C16 pad 2: VCC -> 5V_L
- C17 pad 1: GND -> GND_L
- C17 pad 2: VCC -> 5V_L
- C18 pad 1: GND -> GND_L
- C18 pad 2: VCC -> 5V_L
- C19 pad 1: GND -> GND_L
- C19 pad 2: VCC -> 5V_L
- C2 pad 1: VDD -> 5V_R
- C2 pad 2: GNDA -> GND_R
- C20 pad 1: GNDA -> GND_R
- C20 pad 2: VDD -> 5V_R
- C21 pad 1: VDD -> 5V_R
- C21 pad 2: GNDA -> GND_R
- C22 pad 1: GNDA -> GND_R
- C22 pad 2: VDD -> 5V_R
- C23 pad 1: GNDA -> GND_R
- C23 pad 2: VDD -> 5V_R
- C24 pad 1: VDD -> 5V_R
- C24 pad 2: GNDA -> GND_R
- C25 pad 1: GNDA -> GND_R
- C25 pad 2: VDD -> 5V_R
- C26 pad 1: VDD -> Net-(Q2B-G)
- C26 pad 2: GNDA -> GND_L
- C27 pad 1: VDD -> 5V_R
- C27 pad 2: GNDA -> GND_R
- C28 pad 1: GNDA -> GND_R
- C28 pad 2: VDD -> 5V_R
- C29 pad 1: GNDA -> +5V_L
- C29 pad 2: VDD -> GND
- C30 pad 1: GNDA -> GND
- C30 pad 2: VDD -> Net-(U4-XTAL_IN)
- C31 pad 1: VDD -> 5V_R
- C31 pad 2: GNDA -> GND_R
- C32 pad 1: VDD -> 5V_R
- C32 pad 2: GNDA -> GND_R
- C33 pad 1: VDD -> 5V_R
- C33 pad 2: GNDA -> GND_R
- C34 pad 1: VDD -> 5V_R
- C34 pad 2: GNDA -> GND_R
- C35 pad 1: VDD -> 5V_R
- C35 pad 2: GNDA -> GND_R
- C36 pad 1: VDD -> 5V_R
- C36 pad 2: GNDA -> GND_R
- C37 pad 1: VDD -> 5V_R
- C37 pad 2: GNDA -> GND_R
- C38 pad 1: VDD -> GND
- C38 pad 2: GNDA -> Net-(C38-Pad2)
- C39 pad 1: VDD -> GND
- C39 pad 2: GNDA -> +3V3_L
- C40 pad 1: VDD -> GND
- C40 pad 2: GNDA -> +1V1_L
- C41 pad 1: VCC -> 5V_L
- C41 pad 2: GND -> GND_L
- C42 pad 1: VCC -> 5V_L
- C42 pad 2: GND -> GND_L
- C43 pad 1: VCC -> 5V_L
- C43 pad 2: GND -> GND_L
- C44 pad 1: VCC -> 5V_L
- C44 pad 2: GND -> GND_L
- C45 pad 1: VCC -> 5V_L
- C45 pad 2: GND -> GND_L
- C46 pad 1: VCC -> 5V_L
- C46 pad 2: GND -> GND_L
- C47 pad 1: VCC -> 5V_L
- C47 pad 2: GND -> GND_L
- C48 pad 1: VDD -> 5V_R
- C48 pad 2: GNDA -> GND_R
- C49 pad 1: VDD -> 5V_R
- C49 pad 2: GNDA -> GND_R
- C5 pad 1: VDD -> VBUS_L
- C5 pad 2: GNDA -> GND
- C50 pad 1: VDD -> 5V_R
- C50 pad 2: GNDA -> GND_R
- C51 pad 1: VDD -> 5V_R
- C51 pad 2: GNDA -> GND_R
- C52 pad 1: VDD -> 5V_R
- C52 pad 2: GNDA -> GND_R
- C53 pad 1: VDD -> 5V_R
- C53 pad 2: GNDA -> GND_R
- C54 pad 1: VDD -> 5V_R
- C54 pad 2: GNDA -> GND_R
- C55 pad 1: VDD -> 5V_R
- C55 pad 2: GNDA -> GND_R
- C56 pad 1: VDD -> +3V3_L
- C56 pad 2: GNDA -> GND
- C57 pad 1: VDD -> +3V3_L
- C57 pad 2: GNDA -> GND
- C58 pad 1: VDD -> +3V3_L
- C58 pad 2: GNDA -> GND
- C59 pad 1: VCC -> 5V_L
- C59 pad 2: GND -> GND_L
- C60 pad 1: VCC -> 5V_L
- C60 pad 2: GND -> GND_L
- C61 pad 1: VCC -> 5V_L
- C61 pad 2: GND -> GND_L
- C62 pad 1: VCC -> 5V_L
- C62 pad 2: GND -> GND_L
- C63 pad 1: VCC -> 5V_L
- C63 pad 2: GND -> GND_L
- C64 pad 1: VCC -> 5V_L
- C64 pad 2: GND -> GND_L
- C65 pad 1: VDD -> 5V_R
- C65 pad 2: GNDA -> GND_R
- C66 pad 1: VDD -> 5V_R
- C66 pad 2: GNDA -> GND_R
- C67 pad 1: VDD -> 5V_R
- C67 pad 2: GNDA -> GND_R
- C68 pad 1: VDD -> 5V_R
- C68 pad 2: GNDA -> GND_R
- C69 pad 1: VDD -> 5V_R
- C69 pad 2: GNDA -> GND_R
- C7 pad 1: GND -> GND_L
- C7 pad 2: VCC -> 5V_L
- C70 pad 1: VDD -> 5V_R
- C70 pad 2: GNDA -> GND_R
- C71 pad 1: VDD -> 5V_R
- C71 pad 2: GNDA -> GND_R
- C72 pad 1: VCC -> 5V_L
- C72 pad 2: GND -> GND_L
- C73 pad 1: VCC -> 5V_L
- C73 pad 2: GND -> GND_L
- C74 pad 1: VCC -> 5V_L
- C74 pad 2: GND -> GND_L
- C75 pad 1: VCC -> 5V_L
- C75 pad 2: GND -> GND_L
- C76 pad 1: VCC -> 5V_L
- C76 pad 2: GND -> GND_L
- C77 pad 1: VCC -> 5V_L
- C77 pad 2: GND -> GND_L
- C78 pad 1: VCC -> 5V_L
- C78 pad 2: GND -> GND_L
- C79 pad 1: VDD -> 5V_R
- C79 pad 2: GNDA -> GND_R
- C8 pad 1: GND -> GND_L
- C8 pad 2: VCC -> 5V_L
- C80 pad 1: VDD -> 5V_R
- C80 pad 2: GNDA -> GND_R
- C81 pad 1: VDD -> 5V_R
- C81 pad 2: GNDA -> GND_R
- C82 pad 1: VDD -> 5V_R
- C82 pad 2: GNDA -> GND_R
- C83 pad 1: VDD -> 5V_R
- C83 pad 2: GNDA -> GND_R
- C84 pad 1: VDD -> 5V_R
- C84 pad 2: GNDA -> GND_R
- C85 pad 1: VDD -> +3V3_L
- C85 pad 2: GNDA -> GND
- C86 pad 1: VCC -> 5V_L
- C86 pad 2: GND -> GND_L
- C87 pad 1: VCC -> 5V_L
- C87 pad 2: GND -> GND_L
- C88 pad 1: VCC -> 5V_L
- C88 pad 2: GND -> GND_L
- C89 pad 1: VCC -> 5V_L
- C89 pad 2: GND -> GND_L
- C9 pad 1: GND -> GND_L
- C9 pad 2: VCC -> 5V_L
- C90 pad 1: VCC -> 5V_L
- C90 pad 2: GND -> GND_L
- C91 pad 1: VDD -> 5V_R
- C91 pad 2: GNDA -> GND_R
- C92 pad 1: VDD -> 5V_R
- C92 pad 2: GNDA -> GND_R
- C93 pad 1: VDD -> 5V_R
- C93 pad 2: GNDA -> GND_R
- C94 pad 1: VDD -> 5V_R
- C94 pad 2: GNDA -> GND_R
- C95 pad 1: VDD -> 5V_R
- C95 pad 2: GNDA -> GND_R
- C96 pad 1: VDD -> +3V3_L
- C96 pad 2: GNDA -> GND
- C97 pad 1: VDD -> +3V3_L
- C97 pad 2: GNDA -> GND
- C98 pad 1: VDD -> +1V1_L
- C98 pad 2: GNDA -> GND
- C99 pad 1: VCC -> 5V_L
- C99 pad 2: GND -> GND_L
- J1 pad 1: VDD -> unconnected-(J1-A-Pad1)
- J1 pad 2: GNDA -> unconnected-(J1-B-Pad2)
- J1 pad 3: Net-(J1-Pad3) -> unconnected-(J1-C-Pad3)
- J2 pad 1: VCC -> +5V_L
- J2 pad 2: GND -> GND_L
- J2 pad 3: Net-(J2-Pad3) -> unconnected-(J2-C-Pad3)
- LED1 pad 1: VDD -> 5V_R
- LED1 pad 3: GNDA -> GND_R
- LED10 pad 1: VCC -> 5V_L
- LED10 pad 3: GND -> GND_L
- LED100 pad 1: VCC -> 5V_L
- LED100 pad 3: GND -> GND_L
- LED101 pad 1: VCC -> 5V_L
- LED101 pad 3: GND -> GND_L
- LED102 pad 1: VCC -> 5V_L
- LED102 pad 3: GND -> GND_L
- LED103 pad 1: VCC -> 5V_L
- LED103 pad 2: Net-(LED103-Pad2) -> unconnected-(LED103-DOUT-Pad2)
- LED103 pad 3: GND -> GND_L
- LED104 pad 1: VDD -> 5V_R
- LED104 pad 3: GNDA -> GND_R
- LED11 pad 1: VCC -> 5V_L
- LED11 pad 3: GND -> GND_L
- LED12 pad 1: VCC -> 5V_L
- LED12 pad 3: GND -> GND_L
- LED13 pad 1: VCC -> 5V_L
- LED13 pad 3: GND -> GND_L
- LED14 pad 1: VDD -> 5V_R
- LED14 pad 3: GNDA -> GND_R
- LED15 pad 1: VDD -> 5V_R
- LED15 pad 3: GNDA -> GND_R
- LED16 pad 1: VDD -> 5V_R
- LED16 pad 3: GNDA -> GND_R
- LED17 pad 1: VDD -> 5V_R
- LED17 pad 3: GNDA -> GND_R
- LED18 pad 1: VDD -> 5V_R
- LED18 pad 3: GNDA -> GND_R
- LED19 pad 1: VDD -> 5V_R
- LED19 pad 3: GNDA -> GND_R
- LED2 pad 1: VDD -> 5V_R
- LED2 pad 2: Net-(LED2-Pad2) -> Net-(LED2-DOUT)
- LED2 pad 3: GNDA -> GND_R
- LED20 pad 1: VDD -> 5V_R
- LED20 pad 3: GNDA -> GND_R
- LED20 pad 4: Net-(LED20-Pad4) -> Net-(LED20-DIN)
- LED22 pad 1: VDD -> 5V_R
- LED22 pad 2: Net-(LED21-Pad4) -> Net-(LED20-DIN)
- LED22 pad 3: GNDA -> GND_R
- LED23 pad 1: VDD -> 5V_R
- LED23 pad 3: GNDA -> GND_R
- LED23 pad 4: Net-(LED23-Pad4) -> Net-(LED23-DIN)
- LED26 pad 1: VCC -> 5V_L
- LED26 pad 3: GND -> GND_L
- LED27 pad 1: VCC -> 5V_L
- LED27 pad 3: GND -> GND_L
- LED28 pad 1: VCC -> 5V_L
- LED28 pad 3: GND -> GND_L
- LED29 pad 1: VCC -> 5V_L
- LED29 pad 3: GND -> GND_L
- LED30 pad 1: VCC -> 5V_L
- LED30 pad 3: GND -> GND_L
- LED31 pad 1: VDD -> 5V_R
- LED31 pad 3: GNDA -> GND_R
- LED32 pad 1: VDD -> 5V_R
- LED32 pad 3: GNDA -> GND_R
- LED33 pad 1: VDD -> 5V_R
- LED33 pad 3: GNDA -> GND_R
- LED34 pad 1: VDD -> 5V_R
- LED34 pad 3: GNDA -> GND_R
- LED35 pad 1: VDD -> 5V_R
- LED35 pad 3: GNDA -> GND_R
- LED36 pad 1: VDD -> 5V_R
- LED36 pad 3: GNDA -> GND_R
- LED37 pad 1: VDD -> 5V_R
- LED37 pad 3: GNDA -> Net-(LED37-VSS)
- LED41 pad 1: VCC -> 5V_L
- LED41 pad 3: GND -> GND_L
- LED42 pad 1: VCC -> 5V_L
- LED42 pad 3: GND -> GND_L
- LED43 pad 1: VCC -> 5V_L
- LED43 pad 3: GND -> GND_L
- LED44 pad 1: VCC -> 5V_L
- LED44 pad 3: GND -> GND_L
- LED45 pad 1: VCC -> 5V_L
- LED45 pad 3: GND -> GND_L
- LED46 pad 1: VCC -> 5V_L
- LED46 pad 3: GND -> GND_L
- LED47 pad 1: VCC -> 5V_L
- LED47 pad 3: GND -> GND_L
- LED48 pad 1: VDD -> 5V_R
- LED48 pad 3: GNDA -> GND_R
- LED49 pad 1: VDD -> 5V_R
- LED49 pad 3: GNDA -> GND_R
- LED50 pad 1: VDD -> 5V_R
- LED50 pad 3: GNDA -> GND_R
- LED51 pad 1: VDD -> 5V_R
- LED51 pad 3: GNDA -> GND_R
- LED52 pad 1: VDD -> 5V_R
- LED52 pad 3: GNDA -> GND_R
- LED53 pad 1: VDD -> 5V_R
- LED53 pad 3: GNDA -> GND_R
- LED54 pad 1: VDD -> 5V_R
- LED54 pad 3: GNDA -> GND_R
- LED55 pad 1: VDD -> 5V_R
- LED55 pad 3: GNDA -> Net-(LED37-VSS)
- LED59 pad 1: VCC -> 5V_L
- LED59 pad 3: GND -> GND_L
- LED60 pad 1: VCC -> 5V_L
- LED60 pad 3: GND -> GND_L
- LED61 pad 1: VCC -> 5V_L
- LED61 pad 3: GND -> GND_L
- LED62 pad 1: VCC -> 5V_L
- LED62 pad 3: GND -> GND_L
- LED63 pad 1: VCC -> 5V_L
- LED63 pad 3: GND -> GND_L
- LED64 pad 1: VCC -> 5V_L
- LED64 pad 3: GND -> GND_L
- LED65 pad 1: VDD -> 5V_R
- LED65 pad 3: GNDA -> GND_R
- LED66 pad 1: VDD -> 5V_R
- LED66 pad 3: GNDA -> GND_R
- LED67 pad 1: VDD -> 5V_R
- LED67 pad 3: GNDA -> GND_R
- LED68 pad 1: VDD -> 5V_R
- LED68 pad 3: GNDA -> GND_R
- LED69 pad 1: VDD -> 5V_R
- LED69 pad 3: GNDA -> GND_R
- LED7 pad 1: VCC -> 5V_L
- LED7 pad 3: GND -> GND_L
- LED70 pad 1: VDD -> 5V_R
- LED70 pad 3: GNDA -> GND_R
- LED71 pad 1: VDD -> 5V_R
- LED71 pad 3: GNDA -> GND_R
- LED72 pad 1: VCC -> 5V_L
- LED72 pad 3: GND -> GND_L
- LED73 pad 1: VCC -> 5V_L
- LED73 pad 3: GND -> GND_L
- LED74 pad 1: VCC -> 5V_L
- LED74 pad 3: GND -> GND_L
- LED75 pad 1: VCC -> 5V_L
- LED75 pad 3: GND -> GND_L
- LED76 pad 1: VCC -> 5V_L
- LED76 pad 3: GND -> GND_L
- LED77 pad 1: VCC -> 5V_L
- LED77 pad 3: GND -> GND_L
- LED78 pad 1: VCC -> 5V_L
- LED78 pad 3: GND -> GND_L
- LED79 pad 1: VDD -> 5V_R
- LED79 pad 3: GNDA -> GND_R
- LED8 pad 1: VCC -> 5V_L
- LED8 pad 3: GND -> GND_L
- LED80 pad 1: VDD -> 5V_R
- LED80 pad 3: GNDA -> GND_R
- LED81 pad 1: VDD -> 5V_R
- LED81 pad 3: GNDA -> GND_R
- LED82 pad 1: VDD -> 5V_R
- LED82 pad 3: GNDA -> GND_R
- LED83 pad 1: VDD -> 5V_R
- LED83 pad 3: GNDA -> GND_R
- LED84 pad 1: VDD -> 5V_R
- LED84 pad 3: GNDA -> GND_R
- LED86 pad 1: VCC -> 5V_L
- LED86 pad 3: GND -> GND_L
- LED87 pad 1: VCC -> 5V_L
- LED87 pad 3: GND -> GND_L
- LED88 pad 1: VCC -> 5V_L
- LED88 pad 3: GND -> GND_L
- LED89 pad 1: VCC -> 5V_L
- LED89 pad 3: GND -> GND_L
- LED9 pad 1: VCC -> 5V_L
- LED9 pad 3: GND -> GND_L
- LED90 pad 1: VCC -> 5V_L
- LED90 pad 3: GND -> GND_L
- LED91 pad 1: VDD -> 5V_R
- LED91 pad 2: Net-(LED91-Pad2) -> unconnected-(LED91-DOUT-Pad2)
- LED91 pad 3: GNDA -> GND_R
- LED92 pad 1: VDD -> 5V_R
- LED92 pad 3: GNDA -> GND_R
- LED93 pad 1: VDD -> 5V_R
- LED93 pad 3: GNDA -> GND_R
- LED94 pad 1: VDD -> 5V_R
- LED94 pad 3: GNDA -> GND_R
- LED95 pad 1: VDD -> 5V_R
- LED95 pad 3: GNDA -> Net-(LED37-VSS)
- LED95 pad 4: Net-(LED95-Pad4) -> unconnected-(LED95-DIN-Pad4)
- LED99 pad 1: VCC -> 5V_L
- LED99 pad 3: GND -> GND_L
- OL1 pad 3: VDD -> 5V_R
- OL1 pad 4: GNDA -> GND_R
- OL2 pad 3: VCC -> +5V_L
- OL2 pad 4: GND -> GND_L
- R1 pad 1: Net-(LED25-Pad4) -> Net-(LED23-DIN)
- RSW1 pad 2: GNDA -> GND_R
Routing:
- net VDD: track 1623.1 -> 0.00 mm, vias 39 -> 0
- net GNDA: track 1503.2 -> 0.00 mm, vias 6 -> 0
- net VCC: track 1097.1 -> 0.00 mm, vias 31 -> 0
- net GND: track 969.4 -> 0.00 mm, vias 6 -> 0
- net col0_R: track 338.2 -> 0.00 mm, vias 8 -> 0
- net row1_R: track 335.2 -> 0.00 mm
- net row4_R: track 323.6 -> 0.00 mm, vias 1 -> 0
- net row3_R: track 321.9 -> 0.00 mm, vias 1 -> 0
- net row2_R: track 314.6 -> 0.00 mm, vias 1 -> 0
- net col1_R: track 312.4 -> 0.00 mm, vias 6 -> 0
- net row0_R: track 310.3 -> 0.00 mm
- net col6_L: track 309.6 -> 0.00 mm, vias 10 -> 0
- net col2_R: track 301.7 -> 0.00 mm, vias 6 -> 0
- net col3_R: track 287.8 -> 0.00 mm, vias 8 -> 0
- net col4_R: track 269.0 -> 0.00 mm, vias 8 -> 0
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Other:
- board size 405.8 x 120.8 mm -> 333.6 x 107.9 mm
- copper layers 2 -> 4
- rule pad_to_mask_clearance: 0.2 -> 0

Commit message: flipped usb c
Parts:
- FB1, J5, R7, R8: moved to B.Cu
- J2: moved to F.Cu
- moved C3 154.2 mm to (339.0, 60.0)
- moved FB1 135.2 mm to (50.0, 32.9), turned to -90 degrees
- moved LED3 134.3 mm to (311.9, 55.2)
- moved R7 132.8 mm to (53.1, 38.0), turned to 90 degrees
- moved R8 129.4 mm to (56.1, 38.0), turned to 90 degrees
- moved LED3 129.2 mm to (438.6, 79.5)
- moved C4 125.6 mm to (321.0, 21.6)
- moved C4 125.6 mm to (475.5, 74.0)
- moved LED4 122.7 mm to (468.7, 64.7)
- moved LED4 122.7 mm to (308.6, 22.1)
- moved C21 119.7 mm to (315.9, 17.7)
- moved J4 47.0 mm to (333.6, 25.2), turned to 180 degrees
- turned J5 to 0 degrees
Routing:
- net VBUS_L: track 5.11 -> 10.3 mm
- net /PORT+: track 3.61 -> 0.00 mm, vias 2 -> 0
- net /PORT-: track 4.85 -> 2.31 mm
- net Net-(J5-CC2): track 0.00 -> 1.46 mm
- net Net-(J5-SHIELD): track 0.00 -> 1.43 mm
- net Net-(J5-CC1): track 0.00 -> 1.43 mm
- net GND: track 0.00 -> 0.38 mm, vias 0 -> 1
Other:
- board size 333.6 x 107.9 mm -> 333.6 x 103.7 mm

Commit message: more trace work
Parts:
- removed OL1, OL2: OLED, onigaku:OLED_v2
- removed R3: 4.7k, Resistor_SMD:R_0805_2012Metric_Pad1.20x1.40mm_HandSolder
- J4, TP1, TP2: moved to B.Cu
- moved R2 117.5 mm to (161.8, 68.7), turned to 0 degrees
- moved TP1 74.1 mm to (170.6, 77.5)
- moved TP2 71.2 mm to (171.5, 77.5)
- moved J4 9.71 mm to (326.7, 32.0), turned to 0 degrees
- moved FB1 8.65 mm to (58.7, 32.8)
- moved J1 1.97 mm to (205.9, 35.8)
- moved R7 0.06 mm to (53.0, 38.0)
Connections:
- C10 pad 2: 5V_L -> +5V_L
- C100 pad 1: 5V_L -> +5V_L
- C101 pad 1: 5V_L -> +5V_L
- C102 pad 1: 5V_L -> +5V_L
- C103 pad 1: 5V_L -> +5V_L
- C105 pad 2: GND -> GND_L
- C106 pad 2: GND -> GND_L
- C11 pad 2: 5V_L -> +5V_L
- C12 pad 1: 5V_L -> +5V_L
- C13 pad 2: 5V_L -> +5V_L
- C15 pad 2: 5V_L -> +5V_L
- C16 pad 2: 5V_L -> +5V_L
- C17 pad 2: 5V_L -> +5V_L
- C18 pad 2: 5V_L -> +5V_L
- C19 pad 2: 5V_L -> +5V_L
- C29 pad 2: GND -> GND_L
- C39 pad 1: GND -> GND_L
- C40 pad 1: GND -> GND_L
- C41 pad 1: 5V_L -> +5V_L
- C42 pad 1: 5V_L -> +5V_L
- C43 pad 1: 5V_L -> +5V_L
- C44 pad 1: 5V_L -> +5V_L
- C45 pad 1: 5V_L -> +5V_L
- C46 pad 1: 5V_L -> +5V_L
- C47 pad 1: 5V_L -> +5V_L
- C5 pad 2: GND -> GND_L
- C56 pad 2: GND -> GND_L
- C57 pad 2: GND -> GND_L
- C58 pad 2: GND -> GND_L
- C59 pad 1: 5V_L -> +5V_L
- C5b1 pad 2: GND -> GND_L
- C60 pad 1: 5V_L -> +5V_L
- C61 pad 1: 5V_L -> +5V_L
- C62 pad 1: 5V_L -> +5V_L
- C63 pad 1: 5V_L -> +5V_L
- C64 pad 1: 5V_L -> +5V_L
- C6_A1 pad 2: GND -> GND_L
- C7 pad 2: 5V_L -> +5V_L
- C72 pad 1: 5V_L -> +5V_L
- C73 pad 1: 5V_L -> +5V_L
- C74 pad 1: 5V_L -> +5V_L
- C75 pad 1: 5V_L -> +5V_L
- C76 pad 1: 5V_L -> +5V_L
- C77 pad 1: 5V_L -> +5V_L
- C78 pad 1: 5V_L -> +5V_L
- C8 pad 2: 5V_L -> +5V_L
- C85 pad 2: GND -> GND_L
- C86 pad 1: 5V_L -> +5V_L
- C87 pad 1: 5V_L -> +5V_L
- C88 pad 1: 5V_L -> +5V_L
- C89 pad 1: 5V_L -> +5V_L
- C9 pad 2: 5V_L -> +5V_L
- C90 pad 1: 5V_L -> +5V_L
- C96 pad 2: GND -> GND_L
- C97 pad 2: GND -> GND_L
- C98 pad 2: GND -> GND_L
- C99 pad 1: 5V_L -> +5V_L
- FB1 pad 2: GND -> GND_L
- J5 pad A1: GND -> GND_L
- J5 pad A12: GND -> GND_L
- J5 pad B1: GND -> GND_L
- J5 pad B12: GND -> GND_L
- LED10 pad 1: 5V_L -> +5V_L
- LED100 pad 1: 5V_L -> +5V_L
- LED101 pad 1: 5V_L -> +5V_L
- LED102 pad 1: 5V_L -> +5V_L
- LED103 pad 1: 5V_L -> +5V_L
- LED11 pad 1: 5V_L -> +5V_L
- LED12 pad 1: 5V_L -> +5V_L
- LED13 pad 1: 5V_L -> +5V_L
- LED26 pad 1: 5V_L -> +5V_L
- LED27 pad 1: 5V_L -> +5V_L
- LED28 pad 1: 5V_L -> +5V_L
- LED29 pad 1: 5V_L -> +5V_L
- LED30 pad 1: 5V_L -> +5V_L
- LED41 pad 1: 5V_L -> +5V_L
- LED42 pad 1: 5V_L -> +5V_L
- LED43 pad 1: 5V_L -> +5V_L
- LED44 pad 1: 5V_L -> +5V_L
- LED45 pad 1: 5V_L -> +5V_L
- LED46 pad 1: 5V_L -> +5V_L
- LED47 pad 1: 5V_L -> +5V_L
- LED59 pad 1: 5V_L -> +5V_L
- LED60 pad 1: 5V_L -> +5V_L
- LED61 pad 1: 5V_L -> +5V_L
- LED62 pad 1: 5V_L -> +5V_L
- LED63 pad 1: 5V_L -> +5V_L
- LED64 pad 1: 5V_L -> +5V_L
- LED7 pad 1: 5V_L -> +5V_L
- LED72 pad 1: 5V_L -> +5V_L
- LED73 pad 1: 5V_L -> +5V_L
- LED74 pad 1: 5V_L -> +5V_L
- LED75 pad 1: 5V_L -> +5V_L
- LED76 pad 1: 5V_L -> +5V_L
- LED77 pad 1: 5V_L -> +5V_L
- LED78 pad 1: 5V_L -> +5V_L
- LED8 pad 1: 5V_L -> +5V_L
- LED86 pad 1: 5V_L -> +5V_L
- LED87 pad 1: 5V_L -> +5V_L
- LED88 pad 1: 5V_L -> +5V_L
- LED89 pad 1: 5V_L -> +5V_L
- LED9 pad 1: 5V_L -> +5V_L
- LED90 pad 1: 5V_L -> +5V_L
- LED99 pad 1: 5V_L -> +5V_L
- R10 pad 2: GND -> GND_L
- R15 pad 2: GND -> GND_L
- R7 pad 1: GND -> GND_L
- R8 pad 1: GND -> GND_L
- U2 pad 2: GND -> GND_L
- U2 pad 5: GND -> GND_L
- U3 pad 4: GND -> GND_L
- U3 pad 9: GND -> GND_L
- U4 pad 57: GND -> GND_L
- U5 pad 2: GND -> GND_L
Routing:
- net +5V_L: track 2.84 -> 943.5 mm, vias 3 -> 89
- net VBUS_L: track 10.3 -> 162.7 mm
- net Net-(LED26-DIN): track 0.00 -> 116.6 mm, vias 0 -> 2
- net Net-(LED42-DIN): track 0.00 -> 63.4 mm, vias 0 -> 2
- net Net-(LED72-DOUT): track 0.00 -> 49.4 mm, vias 0 -> 2
- net Net-(LED102-DOUT): track 0.00 -> 44.2 mm, vias 0 -> 2
- net Net-(LED75-DIN): track 0.00 -> 42.3 mm, vias 0 -> 2
- net Net-(LED7-DIN): track 0.00 -> 42.1 mm, vias 0 -> 2
- net Net-(LED103-DIN): track 0.00 -> 40.4 mm, vias 0 -> 2
- net Net-(LED47-DOUT): track 0.00 -> 39.7 mm, vias 0 -> 2
- net Net-(LED10-DOUT): track 0.00 -> 38.3 mm, vias 0 -> 2
- net Net-(LED45-DOUT): track 0.00 -> 37.2 mm, vias 0 -> 2
- net Net-(LED8-DIN): track 0.00 -> 36.9 mm, vias 0 -> 2
- net Net-(LED41-DOUT): track 0.00 -> 36.6 mm, vias 0 -> 2
- net Net-(LED43-DOUT): track 0.00 -> 35.9 mm, vias 0 -> 2
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- added copper zone on In1.Cu, net +3V3_L
- added copper zone on B.Cu, net GND_L
- added copper zone on F.Cu, net GND_L
Other:
- board size 333.6 x 103.7 mm -> 333.6 x 103.8 mm

Commit message: more tracing
Parts:
- moved C96 2.44 mm to (163.7, 78.2), turned to -90 degrees
Routing:
- net row4_L: track 0.00 -> 178.9 mm, vias 0 -> 6
- net row0_L: track 0.00 -> 155.7 mm
- net row3_L: track 0.00 -> 137.8 mm, vias 0 -> 7
- net row1_L: track 0.00 -> 137.5 mm, vias 0 -> 8
- net col0_L: track 0.00 -> 104.5 mm, vias 0 -> 2
- net row2_L: track 0.00 -> 101.3 mm, vias 0 -> 8
- net col1_L: track 0.00 -> 95.0 mm, vias 0 -> 4
- net Net-(LED103-DIN): track 40.4 -> 45.0 mm, vias 2 -> 3
- net Net-(D_47-A): track 0.00 -> 4.04 mm
- net Net-(D_46-A): track 0.00 -> 4.04 mm
- net Net-(D_45-A): track 0.00 -> 4.04 mm
- net Net-(D_44-A): track 0.00 -> 4.04 mm
- net Net-(D_43-A): track 0.00 -> 4.04 mm
- net Net-(LED100-DOUT): track 31.2 -> 35.0 mm, vias 2 -> 4
- net +3V3_L: track 22.4 -> 24.6 mm
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