File: umiko.kicad_pcb (KiCad board)
At the start: 4 copper layers, 333.6 x 103.8 mm, 370 parts, among them J1 MJ-4PP-9, J2 MJ-4PP-9, J4 USB_C_Receptacle_USB2.0_16P_T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, J5 USB_C_Receptacle_USB2.0, Q1 2N7002VC-, Q2 2N7002VC-, SW1 SWITCH, U1 USBLC6-2P6, U2 TLV75533PDQNR, U3 W25Q128JVPIQ, U4 RP2040, U5 74LVC1T45, Y1 12MHz

Commit message: more tracin
Parts:
- moved C97 0.29 mm to (166.5, 70.2)
Connections:
- C30 pad 1: GND -> GND_L
- C38 pad 1: GND -> GND_L
- R17 pad 2: GND -> GND_L
- U4 pad 19: GND -> GND_L
- Y1 pad 4: GND -> GND_L
Routing:
- net col3_L: track 0.00 -> 196.1 mm, vias 4 -> 3
- net col2_L: track 0.00 -> 191.2 mm, vias 4 -> 3
- net col4_L: track 0.00 -> 154.6 mm, vias 2 -> 3
- net /PORT+: track 0.00 -> 144.0 mm, vias 0 -> 2
- net /PORT-: track 2.31 -> 145.9 mm, vias 1 -> 2
- net col6_L: track 0.00 -> 123.7 mm, vias 5 -> 3
- net col1_L: track 95.0 -> 216.7 mm, vias 4 -> 9
- net col0_L: track 104.5 -> 222.9 mm, vias 2 -> 4
- net col5_L: track 0.00 -> 106.0 mm
- net data_L: track 0.84 -> 43.7 mm
- net Net-(Q1A-D): track 3.48 -> 34.8 mm, vias 2 -> 3
- net row2_L: track 101.3 -> 127.5 mm
- net +1V1_L: track 4.36 -> 17.1 mm
- net /QSPI_SD3: track 0.00 -> 12.0 mm, vias 0 -> 2
- net /QSPI_CLK: track 0.00 -> 11.8 mm, vias 0 -> 2
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
Commit message: left side first pass
Parts:
- removed JP1: SolderJumper_2_Open, Jumper:SolderJumper-2_P1.3mm_Open_TrianglePad1.0x1.5mm
Connections:
- D1 pad 2: Net-(D1-A) -> +3V3_L
- U1 pad 2: GND -> GND_L
- U4 pad 19: GND_L -> GND
Routing:
- net data_L: track 43.7 -> 45.9 mm
- net /QSPI_SD1: track 5.42 -> 7.38 mm
- net Net-(D1-A): track 1.62 -> 0.00 mm, vias 2 -> 0
- net /RGB_DO: track 16.3 -> 17.8 mm
- net GND_L: track 4.43 -> 5.86 mm, vias 7 -> 20
- net +5V_L: track 944.4 -> 945.1 mm
- net +3V3_L: vias 14 -> 15

Commit message: more tracing
Routing:
- net Net-(LED100-DOUT): track 35.0 -> 45.9 mm, vias 4 -> 3
- net Net-(LED72-DOUT): track 49.4 -> 54.3 mm
- net Net-(LED59-DOUT): track 32.3 -> 37.0 mm, vias 2 -> 5
- net col2_L: track 191.2 -> 194.8 mm
- net Net-(LED11-DIN): track 31.7 -> 35.0 mm, vias 2 -> 3
- net GND_L: track 5.86 -> 8.79 mm, vias 20 -> 22
- net +5V_L: track 945.1 -> 942.3 mm, vias 89 -> 111
- net Net-(LED101-DIN): track 24.2 -> 26.5 mm, vias 2 -> 3
- net Net-(LED42-DIN): track 63.4 -> 65.6 mm, vias 2 -> 4
- net Net-(LED27-DOUT): track 21.5 -> 23.6 mm
- net Net-(LED75-DIN): track 42.3 -> 40.3 mm
- net Net-(LED74-DOUT): track 21.8 -> 23.2 mm, vias 2 -> 3
- net data_L: track 45.9 -> 44.6 mm
- net Net-(LED76-DOUT): track 25.2 -> 24.1 mm, vias 2 -> 3
- net Net-(LED28-DOUT): track 30.9 -> 29.8 mm
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
Commit message: moved leds up
Parts:
- added TP1: CLK, PCM_0xcb:TestPoint_Pad_D0.8mm, F.Cu at (168.5, 87.5)
- added TP2: DIO, PCM_0xcb:TestPoint_Pad_D0.8mm, F.Cu at (168.5, 89.3)
- SW_1, SW_18, SW_19, SW_2, SW_20, SW_21, SW_22, SW_23, SW_24, SW_3, SW_35, SW_36, SW_37, SW_38, SW_39, SW_4, SW_40, SW_48, SW_49, SW_5, SW_50, SW_51, SW_52, SW_6: footprint onigaku:CherryMX_Hotswap -> Gateron_KS33_Hotswap:Gateron-KS33-Hotswap-1U
- SW_11, SW_12, SW_13, SW_14, SW_15, SW_16, SW_17, SW_30, SW_31, SW_32, SW_33, SW_34, SW_43, SW_44, SW_45, SW_46, SW_47, SW_56, SW_57, SW_58, SW_59, SW_60: footprint onigaku:CherryMX_Hotswap -> Gateron_KS33_Hotswap:Gateron-KS33-Hotswap-1U; moved to B.Cu
- SW_25: footprint onigaku:CherryMX_Hotswap_1.5u -> Gateron_KS33_Hotswap:Gateron-KS33-Hotswap-1.5U
- SW_29: footprint onigaku:CherryMX_Hotswap_1.5u -> Gateron_KS33_Hotswap:Gateron-KS33-Hotswap-1.5U; moved to B.Cu
- SW_41: footprint onigaku:CherryMX_Hotswap_2.25u_North -> onigaku:Gateron-KS33-2.0-Hotswap-2.25U_stabilized
- SW_42: footprint onigaku:CherryMX_Hotswap_1.75u -> Gateron_KS33_Hotswap:Gateron-KS33-Hotswap-1.75U; moved to B.Cu
- SW_53: footprint onigaku:CherryMX_Hotswap_2.75u_North -> onigaku:Gateron-KS33-2.0-Hotswap-2.75U_stabilized
- SW_55: footprint onigaku:CherryMX_Hotswap_2.25u_North -> onigaku:Gateron-KS33-2.0-Hotswap-2.25U_stabilized; moved to B.Cu
- SW_61: footprint onigaku:CherryMX_Hotswap_2.75u_North_reversed_stabilizers -> onigaku:Gateron-KS33-2.0-Hotswap-2.75U_stabilized
- SW_62, SW_63, SW_64, SW_65: footprint onigaku:CherryMX_Hotswap_1.25u_North -> Gateron_KS33_Hotswap:Gateron-KS33-Hotswap-1.25U
- SW_69, SW_70, SW_71, SW_72: footprint onigaku:CherryMX_Hotswap_1.25u_North -> Gateron_KS33_Hotswap:Gateron-KS33-Hotswap-1.25U; moved to B.Cu
- SW_7: footprint onigaku:CherryMX_Hotswap_2u_North -> Gateron_KS33_Hotswap:Gateron-KS33-Hotswap-2U
- SW_73: footprint onigaku:CherryMX_Hotswap_2.25u_North_reversed_stabilizers -> onigaku:Gateron-KS33-2.0-Hotswap-2.25U_stabilized; moved to B.Cu
- moved D_70 15.6 mm to (78.7, 121.9)
- moved D_58 15.4 mm to (133.5, 102.9)
- moved D_30 15.4 mm to (81.1, 64.8)
- moved D_11 15.4 mm to (52.5, 45.7)
- moved D_43 15.4 mm to (85.8, 83.8)
- moved D_44 15.4 mm to (104.9, 83.8)
- moved D_46 15.4 mm to (143.0, 83.8)
- moved D_57 15.4 mm to (114.4, 102.9)
- moved D_59 15.4 mm to (152.5, 102.9)
- moved D_45 15.4 mm to (123.9, 83.8)
- moved D_47 15.4 mm to (162.0, 83.8)
- moved D_55 15.4 mm to (64.4, 102.9)
- moved D_71 15.4 mm to (102.5, 121.9)
- moved D_34 15.4 mm to (157.3, 64.8)
- moved D_13 15.4 mm to (90.6, 45.7)
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Routing:
- net col2_L: track 194.8 -> 86.1 mm, vias 3 -> 2
- net col1_L: track 216.7 -> 112.5 mm, vias 9 -> 4
- net col6_L: track 123.7 -> 27.8 mm, vias 3 -> 2
- net col5_L: track 105.7 -> 49.7 mm, vias 3 -> 2
- net row1_L: track 137.5 -> 93.2 mm
- net row2_L: track 127.5 -> 88.3 mm
- net col3_L: track 196.1 -> 163.7 mm, vias 3 -> 2
- net Net-(D_12-A): track 4.04 -> 35.8 mm, vias 0 -> 2
- net col4_L: track 154.8 -> 125.1 mm
- net Net-(LED100-DOUT): track 45.9 -> 22.3 mm
- net +5V_L: track 942.3 -> 960.4 mm, vias 111 -> 83
- net Net-(LED102-DOUT): track 44.2 -> 30.3 mm
- net col0_L: track 222.6 -> 236.4 mm
- net Net-(LED75-DIN): track 40.3 -> 28.1 mm
- net row3_L: track 137.8 -> 125.8 mm
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Other:
- outline, holes or cut-outs redrawn
