File: _autosave-umiko.kicad_sch (KiCad schematic)
At the start: 363 parts, among them J1 MJ-4PP-9, J2 MJ-4PP-9, J4 USB_C_Receptacle_USB2.0_16P_T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, J5 USB_C_Receptacle_USB2.0, Q1 2N7002VC-, Q2 2N7002VC-, SW1 SWITCH, U1 USBLC6-2P6, U2 TLV75533PDQNR, U3 W25Q128JVPIQ, U4 RP2040, U5 74LVC1T45, Y1 12MHz

Commit message: left side first pass
Connections:
- net GND: no longer C30.1, C38.1, Y1.4
- net GND_L: now also C30.1, C38.1, Y1.4
Changed lines of the file:
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@@
 			)
 		)
-		(property "Value" "GND"
+		(property "Value" "GND_L"
 			(at 382.27 125.73 0)
 			(effects
