File: umiko.kicad_sch (KiCad schematic)
At the start: 366 parts, among them J1 MJ-4PP-9, J2 MJ-4PP-9, J4 USB_C_Receptacle_USB2.0_16P_T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, J5 USB_C_Receptacle_USB2.0, Q1 2N7002VC-, Q2 2N7002VC-, SW1 SWITCH, U1 USBLC6-2P6, U2 TLV75533PDQNR, U3 W25Q128JVPIQ, U4 RP2040, U5 74LVC1T45, Y1 12MHz

Commit message: more trace work
Parts:
- removed OL1, OL2: OLED, onigaku:OLED_v2, symbol umiko-rescue:OLED-kbd
Connections:
- net 5V_L is gone; now on net +5V_L: C10.2, C100.1, C101.1, C102.1, C103.1, C11.2, C12.1, C13.2, C15.2, C16.2, C17.2, C18.2, C19.2, C41.1, C42.1, C43.1, C44.1, C45.1, C46.1, C47.1, C59.1, C60.1, C61.1, C62.1, C63.1, C64.1, C7.2, C72.1, C73.1, C74.1, C75.1, C76.1, C77.1, C78.1, C8.2, C86.1, C87.1, C88.1, C89.1, C9.2, C90.1, C99.1, LED10.1 (VDD), LED100.1 (VDD), LED101.1 (VDD), LED102.1 (VDD), LED103.1 (VDD), LED11.1 (VDD), LED12.1 (VDD), LED13.1 (VDD), LED26.1 (VDD), LED27.1 (VDD), LED28.1 (VDD), LED29.1 (VDD), LED30.1 (VDD), LED41.1 (VDD), LED42.1 (VDD), LED43.1 (VDD), LED44.1 (VDD), LED45.1 (VDD), LED46.1 (VDD), LED47.1 (VDD), LED59.1 (VDD), LED60.1 (VDD), LED61.1 (VDD), LED62.1 (VDD), LED63.1 (VDD), LED64.1 (VDD), LED7.1 (VDD), LED72.1 (VDD), LED73.1 (VDD), LED74.1 (VDD), LED75.1 (VDD), LED76.1 (VDD), LED77.1 (VDD), LED78.1 (VDD), LED8.1 (VDD), LED86.1 (VDD), LED87.1 (VDD), LED88.1 (VDD), LED89.1 (VDD), LED9.1 (VDD), LED90.1 (VDD), LED99.1 (VDD)
- net GND: no longer C105.2, C106.2, C29.2, C39.1, C40.1, C5.2, C56.2, C57.2, C58.2, C5b1.2, C6_A1.2, C85.2, C96.2, C97.2, C98.2, FB1.2, J5.A1 (GND), J5.A12 (GND), J5.B1 (GND), J5.B12 (GND), R10.2, R15.2, R7.1, R8.1, U2.2 (GND), U2.5 (TP), U3.4 (GND), U3.9 (GND), U4.57 (GND), U5.2 (GND)
- net GND_L: now also C105.2, C106.2, C29.2, C39.1, C40.1, C5.2, C56.2, C57.2, C58.2, C5b1.2, C6_A1.2, C85.2, C96.2, C97.2, C98.2, FB1.2, J5.A1 (GND), J5.A12 (GND), J5.B1 (GND), J5.B12 (GND), R10.2, R15.2, R7.1, R8.1, U2.2 (GND), U2.5 (TP), U3.4 (GND), U3.9 (GND), U4.57 (GND), U5.2 (GND)
Other:
- moved on the sheet: C1, C104, C14, C2, C20, C21, C22, C23, C24, C25, C27, C28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

Commit message: more tracin
Connections:
- net GND: no longer R17.2
- net GND_L: now also R17.2
Changed lines of the file:
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@@
 			)
 		)
-		(property "Value" "GND"
+		(property "Value" "GND_L"
 			(at 485.14 144.78 0)
 			(effects

Commit message: left side first pass
Parts:
- removed JP1: SolderJumper_2_Open, Jumper:SolderJumper-2_P1.3mm_Open_TrianglePad1.0x1.5mm, symbol Jumper:SolderJumper_2_Open
Connections:
- net +3V3_L: now also D1.2 (A)
- net GND: no longer U1.2 (GND)
- net GND_L: now also U1.2 (GND)
Changed lines of the file:
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@@
 	(wire
 		(pts
+			(xy 315.595 78.74) (xy 315.595 86.36)
+		)
+		(stroke
+			(width 0)
+			(type default)
+		)
+	)
+	(wire
+		(pts
 			(xy 775.335 86.36) (xy 775.335 87.63)
 		)
@@
 	)
 	(symbol
-		(lib_id "Jumper:SolderJumper_2_Open")
-		(at 315.595 82.55 270)
-		(unit 1)
-		(exclude_from_sim no)
-		(in_bom no)
-		(on_board yes)
-		(dnp no)
-		(fields_autoplaced yes)
-		(property "Reference" "JP1"
-			(at 318.135 82.5499 90)
-			(effects
-				(font
-					(size 1.27 1.27)
-				)
-				(justify left)
-			)
-		)
-		(property "Value" "SolderJumper_2_Open"
-			(at 313.055 81.2801 90)
-			(effects
-				(font
-					(size 1.27 1.27)
-				)
-				(justify right)
-				(hide yes)
-			)
-		)
-		(property "Footprint" "Jumper:SolderJumper-2_P1.3mm_Open_TrianglePad1.0x1.5mm"
-			(at 315.595 82.55 0)
-			(effects
-				(font
-					(size 1.27 1.27)
-				)
-				(hide yes)
-			)
-		)
-		(property "Datasheet" "~"
-			(at 315.595 82.55 0)
-			(effects
-				(font
-					(size 1.27 1.27)
-				)
-				(hide yes)
-			)
-		)
-		(property "Description" ""
-			(at 315.595 82.55 0)
-			(effects
-				(font
-					(size 1.27 1.27)
-				)
-			)
-		)
-		(property "JLCPCB_CORRECTION" ""
-			(at 315.595 82.55 0)
-			(effects
-				(font
-					(size 1.27 1.27)
-				)
-				(hide yes)
-			)
-		)
-		(property "LCSC" ""
-			(at 315.595 82.55 0)
-			(effects
-				(font
-					(size 1.27 1.27)
-				)
-				(hide yes)
-			)
-		)
-		(pin "1"
-		)
-		(pin "2"
-		)
-		(instances
-			(project "umiko"
-				(path "/4b4aa2f9-db35-4fc9-9772-4a4fa5dd4e1a"
-					(reference "JP1")
-					(unit 1)
-				)
-			)
-		)
-	)
-	(symbol
 		(lib_id "power:PWR_FLAG")
 		(at 343.535 96.52 0)
@@
 			)
 		)
-		(property "Value" "GND"
+		(property "Value" "GND_L"
 			(at 295.275 88.9 0)
 			(effects

Commit message: more tracing
Connections:
- net GND: no longer C30.1, C38.1, Y1.4
- net GND_L: now also C30.1, C38.1, Y1.4
Changed lines of the file:
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@@
 	(generator "eeschema")
 	(generator_version "9.0")
-	(paper "User" 1500.01 450.012)
+	(paper "User" 1000 450.012)
 	(title_block
 		(title "recess")
@@
 				)
 				(justify left)
+				(hide yes)
 			)
 		)
@@
 				)
 				(justify left)
+				(hide yes)
 			)
 		)
@@
 			)
 		)
-		(property "Value" "GND"
+		(property "Value" "GND_L"
 			(at 382.27 125.73 0)
 			(effects

Commit message: moved leds up
Parts:
- SW_1, SW_11, SW_12, SW_13, SW_14, SW_15, SW_16, SW_17, SW_18, SW_19, SW_2, SW_20, SW_21, SW_22, SW_23, SW_24, SW_3, SW_30, SW_31, SW_32, SW_33, SW_34, SW_35, SW_36, SW_37, SW_38, SW_39, SW_4, SW_40, SW_43, SW_44, SW_45, SW_46, SW_47, SW_48, SW_49, SW_5, SW_50, SW_51, SW_52, SW_56, SW_57, SW_58, SW_59, SW_6, SW_60: footprint onigaku:CherryMX_Hotswap -> Gateron_KS33_Hotswap:Gateron-KS33-Hotswap-1U
- SW_25, SW_29: footprint onigaku:CherryMX_Hotswap_1.5u -> Gateron_KS33_Hotswap:Gateron-KS33-Hotswap-1.5U
- SW_41, SW_55: footprint onigaku:CherryMX_Hotswap_2.25u_North -> onigaku:Gateron-KS33-2.0-Hotswap-2.25U_stabilized
- SW_42: footprint onigaku:CherryMX_Hotswap_1.75u -> Gateron_KS33_Hotswap:Gateron-KS33-Hotswap-1.75U
- SW_53: footprint onigaku:CherryMX_Hotswap_2.75u_North -> onigaku:Gateron-KS33-2.0-Hotswap-2.75U_stabilized
- SW_61: footprint onigaku:CherryMX_Hotswap_2.75u_North_reversed_stabilizers -> onigaku:Gateron-KS33-2.0-Hotswap-2.75U_stabilized
- SW_62, SW_63, SW_64, SW_65, SW_69, SW_70, SW_71, SW_72: footprint onigaku:CherryMX_Hotswap_1.25u_North -> Gateron_KS33_Hotswap:Gateron-KS33-Hotswap-1.25U
- SW_7: footprint onigaku:CherryMX_Hotswap_2u_North -> Gateron_KS33_Hotswap:Gateron-KS33-Hotswap-2U
- SW_73: footprint onigaku:CherryMX_Hotswap_2.25u_North_reversed_stabilizers -> onigaku:Gateron-KS33-2.0-Hotswap-2.25U_stabilized

Commit message: moving chips closer
Other:
- moved on the sheet: J1
Changed lines of the file:
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@@
 	)
 	(no_connect
-		(at 603.885 361.315)
+		(at 621.665 192.405)
 	)
 	(no_connect
@@
 	(wire
 		(pts
-			(xy 606.425 365.125) (xy 606.425 363.855)
+			(xy 624.205 196.215) (xy 624.205 194.945)
 		)
 		(stroke
@@
 	(wire
 		(pts
-			(xy 603.885 363.855) (xy 606.425 363.855)
+			(xy 621.665 194.945) (xy 624.205 194.945)
 		)
 		(stroke
@@
 	(global_label "data_R"
 		(shape input)
-		(at 603.885 358.775 0)
+		(at 621.665 189.865 0)
 		(fields_autoplaced yes)
 		(effects
@@
 		)
 		(property "Intersheetrefs" "${INTERSHEET_REFS}"
-			(at 613.3756 358.775 0)
+			(at 631.1556 189.865 0)
 			(effects
 				(font
@@
 	(symbol
 		(lib_id "mj-4pp-9:MJ-4PP-9")
-		(at 589.915 358.775 0)
+		(at 607.695 189.865 0)
 		(unit 1)
 		(exclude_from_sim no)
@@
 		(dnp no)
 		(property "Reference" "J1"
-			(at 589.915 351.155 0)
+			(at 607.695 182.245 0)
 			(effects
 				(font
@@
 		)
 		(property "Value" "MJ-4PP-9"
-			(at 589.915 367.665 0)
+			(at 607.695 198.755 0)
 			(effects
 				(font
@@
 		)
 		(property "Footprint" "mj-4pp-9:MJ-4PP-9"
-			(at 574.675 361.315 0)
+			(at 592.455 192.405 0)
 			(effects
 				(font
@@
 		)
 		(property "Datasheet" ""
-			(at 574.675 361.315 0)
+			(at 592.455 192.405 0)
 			(effects
 				(font
@@
 		)
 		(property "Description" ""
-			(at 589.915 358.775 0)
+			(at 607.695 189.865 0)
 			(effects
 				(font
@@
 	(symbol
 		(lib_id "bakekujira-rescue:GNDA-power")
-		(at 606.425 365.125 0)
+		(at 624.205 196.215 0)
 		(unit 1)
 		(exclude_from_sim no)
@@
 		(dnp no)
 		(property "Reference" "#PWR016"
-			(at 606.425 371.475 0)
+			(at 624.205 202.565 0)
 			(effects
 				(font
@@
 		)
 		(property "Value" "GNDA"
-			(at 606.425 368.935 0)
+			(at 624.205 200.025 0)
 			(effects
 				(font
@@
 		)
 		(property "Footprint" ""
-			(at 606.425 365.125 0)
+			(at 624.205 196.215 0)
 			(effects
 				(font
@@
 		)
 		(property "Datasheet" ""
-			(at 606.425 365.125 0)
+			(at 624.205 196.215 0)
 			(effects
 				(font
@@
 		)
 		(property "Description" ""
-			(at 606.425 365.125 0)
+			(at 624.205 196.215 0)
 			(effects
 				(font
@@
 	(symbol
 		(lib_id "bakekujira-rescue:VDD-power")
-		(at 603.885 354.965 270)
+		(at 621.665 186.055 270)
 		(unit 1)
 		(exclude_from_sim no)
@@
 		(dnp no)
 		(property "Reference" "#PWR0180"
-			(at 600.075 354.965 0)
+			(at 617.855 186.055 0)
 			(effects
 				(font
@@
 		)
 		(property "Value" "VDD"
-			(at 607.695 354.965 0)
+			(at 625.475 186.055 0)
 			(effects
 				(font
@@
 		)
 		(property "Footprint" ""
-			(at 603.885 354.965 0)
+			(at 621.665 186.055 0)
 			(effects
 				(font
@@
 		)
 		(property "Datasheet" ""
-			(at 603.885 354.965 0)
+			(at 621.665 186.055 0)
 			(effects
 				(font
@@
 		)
 		(property "Description" ""
-			(at 603.885 354.965 0)
+			(at 621.665 186.055 0)
 			(effects
 				(font

Commit message: before claude
Parts:
- removed J4: USB_C_Receptacle_USB2.0_16P_TRRS, PCM_marbastlib-various:USB_C_Receptacle_HRO_TYPE-C-31-M-12, symbol Connector:USB_C_Receptacle_USB2.0_16P
- removed RSW1: SW_PUSH, Button_Switch_SMD:SW_SPST_TL3342, symbol umiko-rescue:SW_PUSH-kbd
- added C107, C108, C5b2, C6: 10u, Capacitor_SMD:C_0402_1005Metric, symbol Device:C
- added C109, C110: 15p, Capacitor_SMD:C_0402_1005Metric, symbol Device:C
- added C111, C112: 1u, Capacitor_SMD:C_0402_1005Metric, symbol Device:C
- added C113, C114, C115, C116, C117, C118, C119, C120, C121, C6_A2: 100n, Capacitor_SMD:C_0402_1005Metric, symbol Device:C
- added C6b2: 4.7u, Capacitor_SMD:C_0402_1005Metric, symbol Device:C
- added D4: PMEG2010BELD, PCM_0xcb:SOD882D, symbol Device:D_Schottky
- added D5: Power LED, Diode_SMD:D_0402_1005Metric, symbol Device:LED
- added D6: User LED, Diode_SMD:D_0402_1005Metric, symbol Device:LED
- added F2: 500mA, Fuse:Fuse_0603_1608Metric, symbol Device:Polyfuse_Small
- added FB2: 600R, Resistor_SMD:R_0402_1005Metric, symbol Device:FerriteBead_Small
- added J3: USB_C_Receptacle_USB2.0, PCM_0xcb:USB_C_Receptacle_HRO_TYPE-C-31-M-12, symbol Connector:USB_C_Receptacle_USB2.0
- added Q3, Q4: 2N7002VC-, PCM_0xcb:SOT-563, symbol Transistor_FET:FDG6335N
- added R18, R19, R27: 5.1k, Resistor_SMD:R_0402_1005Metric, symbol Device:R
- added R20, R21, R25, R26: 1k, Resistor_SMD:R_0402_1005Metric, symbol Device:R
- added R22, R28, R3_L2, R3b2, R4b2: 10k, Resistor_SMD:R_0402_1005Metric, symbol Device:R
- added R23, R24: 27, Resistor_SMD:R_0402_1005Metric, symbol Device:R
- added R3, R4, R4_L2: 51k, Resistor_SMD:R_0402_1005Metric, symbol Device:R
- added SW2: SWITCH, PCM_0xcb:1.9x2.8mm SW, symbol Switch:SW_Push
- added TP3: CLK, PCM_0xcb:TestPoint_Pad_D0.8mm, symbol Connector:TestPoint_Small
- added TP4: DIO, PCM_0xcb:TestPoint_Pad_D0.8mm, symbol Connector:TestPoint_Small
- added U10: 74LVC1T45, PCM_0xcb:SOT-563, symbol Logic_LevelTranslator:SN74LVC1T45DRL
- added U6: USBLC6-2P6, Package_TO_SOT_SMD:SOT-666, symbol Power_Protection:USBLC6-2P6
- added U7: TLV75533PDQNR, PCM_0xcb:X2SON-4, symbol 0xcb:LP5907SNX-3.3-NOPB
- added U8: W25Q128JVPIQ, PCM_0xcb:W25Q128JVPIQ, symbol 0xcb:W25Q128JVPIQ
- added U9: RP2040, Package_DFN_QFN:QFN-56-1EP_7x7mm_P0.4mm_EP3.2x3.2mm, symbol 0xcb:RP2040
- added Y2: 12MHz, Crystal:Crystal_SMD_2520-4Pin_2.5x2.0mm, symbol Device:Crystal_GND24_Small
- C105, C106, C56, C57, C58, C6_A1, C85, C96, C97, C98: MPN (none) -> 100nF 10% 10V 0402; MPN  100nF 10% 10V 0402 -> (none)
- C26, C29, C5, C5b1: MPN (none) -> 10uF 20% 10V 0402; MPN  10uF 20% 10V 0402 -> (none)
- C30, C38: MPN (none) -> 15pF 5% 10V; MPN  15pF 5% 10V -> (none)
- C39, C40: MPN (none) -> 1uF 20% 10V 0402; MPN  1uF 20% 10V 0402 -> (none)
- C6b1: MPN (none) -> 4.7uF 20% 10V 0402; MPN  4.7uF 20% 10V 0402 -> (none)
- D1: MPN (none) -> B1811URO-20D000113U1930; MPN  B1811URO-20D000113U1930 -> (none)
- D2: MPN (none) -> B1811NB--05D000113U1930; MPN  B1811NB--05D000113U1930 -> (none)
- D3: MPN (none) -> PMEG2010BELD,315; MPN  PMEG2010BELD,315 -> (none)
- F1: MPN (none) -> MF-FSMF050X-2; MPN  MF-FSMF050X-2 -> (none)
- FB1: MPN (none) -> BLM15PX601SN1D; MPN  BLM15PX601SN1D -> (none)
- J5: MPN (none) -> USB4510-03-1-A; MPN  USB4510-03-1-A -> (none)
- Q1, Q2: MPN (none) -> 2N7002VC; MPN  2N7002VC -> (none)
- R10, R14, R15, R9: MPN (none) -> 1k 1% 0402; MPN  1k 1% 0402 -> (none)
- R11, R17, R3_L1, R3b1, R4b1: MPN (none) -> 10k 1% 0402; MPN  10k 1% 0402 -> (none)
- R12, R13: MPN (none) -> 27 1% 0402; MPN  27 1% 0402 -> (none)
- R16, R7, R8: MPN (none) -> 5.1k 1% 0402; MPN  5.1k 1% 0402 -> (none)
- R4_L1, R5, R6: MPN (none) -> 51k 1% 0402; MPN  51k 1% 0402 -> (none)
- SW1: MPN (none) -> EVP-BL2A1B000; MPN  EVP-BL2A1B000 -> (none)
- U1: MPN (none) -> USBLC6-2P6; MPN  USBLC6-2P6 -> (none)
- U2: MPN (none) -> TLV75533PDQNR; MPN  TLV75533PDQNR -> (none)
- U3: MPN (none) -> W25Q128JVPIQ; MPN  W25Q128JVPIQ -> (none)
- U4: MPN (none) -> SC0914(13); MPN  SC0914(13) -> (none)
- U5: MPN (none) -> SN74LVC1T45DRLR; MPN  SN74LVC1T45DRLR -> (none)
- Y1: MPN (none) -> ECS-120-10-36B-CWY-TR3; MPN  ECS-120-10-36B-CWY-TR3 -> (none)
Connections:
- net 5V_R is gone; now on net +5V_R: C1.1, C104.1, C14.1, C2.1, C20.2, C21.1, C22.2, C23.2, C24.1, C25.2, C27.1, C28.2, C3.1, C31.1, C32.1, C33.1, C34.1, C35.1, C36.1, C37.1, C4.1, C48.1, C49.1, C50.1, C51.1, C52.1, C53.1, C54.1, C55.1, C65.1, C66.1, C67.1, C68.1, C69.1, C70.1, C71.1, C79.1, C80.1, C81.1, C82.1, C83.1, C84.1, C91.1, C92.1, C93.1, C94.1, C95.1, LED1.1 (VDD), LED104.1 (VDD), LED14.1 (VDD), LED15.1 (VDD), LED16.1 (VDD), LED17.1 (VDD), LED18.1 (VDD), LED19.1 (VDD), LED2.1 (VDD), LED20.1 (VDD), LED22.1 (VDD), LED23.1 (VDD), LED3.1 (VDD), LED31.1 (VDD), LED32.1 (VDD), LED33.1 (VDD), LED34.1 (VDD), LED35.1 (VDD), LED36.1 (VDD), LED37.1 (VDD), LED4.1 (VDD), LED48.1 (VDD), LED49.1 (VDD), LED50.1 (VDD), LED51.1 (VDD), LED52.1 (VDD), LED53.1 (VDD), LED54.1 (VDD), LED55.1 (VDD), LED65.1 (VDD), LED66.1 (VDD), LED67.1 (VDD), LED68.1 (VDD), LED69.1 (VDD), LED70.1 (VDD), LED71.1 (VDD), LED79.1 (VDD), LED80.1 (VDD), LED81.1 (VDD), LED82.1 (VDD), LED83.1 (VDD), LED84.1 (VDD), LED91.1 (VDD), LED92.1 (VDD), LED93.1 (VDD), LED94.1 (VDD), LED95.1 (VDD)
- net GND is gone; now on net GND_L: U4.19 (TESTEN)
- net col0_R is gone; now on net col0_L: SW_1.1 (COL), SW_18.1 (COL), SW_35.1 (COL), SW_48.1 (COL), SW_61.1 (COL)
- net col1_R is gone; now on net col1_L: SW_19.1 (COL), SW_2.1 (COL), SW_36.1 (COL), SW_49.1 (COL)
- net col2_R is gone; now on net col2_L: SW_20.1 (COL), SW_3.1 (COL), SW_37.1 (COL), SW_50.1 (COL)
- net col3_R is gone; now on net col3_L: SW_21.1 (COL), SW_38.1 (COL), SW_4.1 (COL), SW_51.1 (COL), SW_62.1 (COL)
- net col4_R is gone; now on net col4_L: SW_22.1 (COL), SW_39.1 (COL), SW_5.1 (COL), SW_52.1 (COL), SW_63.1 (COL)
- net col5_R is gone; now on net col5_L: SW_23.1 (COL), SW_40.1 (COL), SW_6.1 (COL)
- net col6_R is gone; now on net col6_L: SW_24.1 (COL), SW_41.1 (COL), SW_53.1 (COL), SW_64.1 (COL)
- net data_R is gone; now on net data_L: J1.4 (D)
- net row0_R is gone; now on net row0_L: D_1.1 (K), D_2.1 (K), D_3.1 (K), D_4.1 (K), D_5.1 (K), D_6.1 (K), D_7.1 (K)
- net row1_R is gone; now on net row1_L: D_18.1 (K), D_19.1 (K), D_20.1 (K), D_21.1 (K), D_22.1 (K), D_23.1 (K), D_24.1 (K), D_25.1 (K)
- net row2_R is gone; now on net row2_L: D_35.1 (K), D_36.1 (K), D_37.1 (K), D_38.1 (K), D_39.1 (K), D_40.1 (K), D_41.1 (K)
- net row3_R is gone; now on net row3_L: D_48.1 (K), D_49.1 (K), D_50.1 (K), D_51.1 (K), D_52.1 (K), D_53.1 (K)
- net row4_R is gone; now on net row4_L: D_61.1 (K), D_62.1 (K), D_63.1 (K), D_64.1 (K), D_65.1 (K)
- net +1V1_L: now also C112.2, C119.1, C121.1, U9.23 (DVDD), U9.45 (VREG_VOUT), U9.50 (DVDD)
- net +3V3_L: now also C111.2, C113.1, C114.1, C115.1, C116.1, C117.1, C118.1, C120.1, C5b2.1, C6_A2.1, D5.2 (A), R22.1, R3_L2.1, R3b2.1, R4b2.1, U10.1 (VCCA), U10.5 (DIR), U7.1 (Vout), U8.8 (VCC), U9.1 (IOVDD), U9.10 (IOVDD), U9.22 (IOVDD), U9.33 (IOVDD), U9.42 (IOVDD), U9.43 (ADC_AVDD), U9.44 (VREG_VIN), U9.48 (USB_VDD), U9.49 (IOVDD)
- net 16: now also U9.27 (GPIO16)
- net 1_RX0: now also U9.3 (GPIO1)
- net 20_SDI: now also U9.31 (GPIO20)
- net 21_CS: now also U9.32 (GPIO21)
- net 22_SCK: now also U9.34 (GPIO22)
- net 23_SDO: now also U9.35 (GPIO23)
- net A0: now also U9.38 (GPIO26/ADC0)
- net A1: now also U9.39 (GPIO27/ADC1)
- net A2: now also U9.40 (GPIO28/ADC2)
- net A3: now also U9.41 (GPIO29/ADC3)
- net BOOT: now also Q4.3 (D), R20.2
- net D+: now also R23.2, U9.47 (D+)
- net D-: now also R24.2, U9.46 (D-)
- net GND_L: now also C108.2, C5b2.2, Q3.4 (S), U6.2 (GND), U7.2 (GND), U7.5 (TP)
- net GND_R: now also J1.2 (B), C107.2, C109.1, C110.1, C111.1, C112.1, C113.2, C114.2, C115.2, C116.2, C117.2, C118.2, C119.2, C120.2, C121.2, C6.2, C6_A2.2, C6b2.2, FB2.2, J3.A1 (GND), J3.A12 (GND), J3.B1 (GND), J3.B12 (GND), Q3.1 (S), Q4.4 (S), R18.1, R19.1, R21.2, R26.2, R28.2, R4.2, SW2.1, U10.2 (GND), U8.4 (GND), U8.9 (GND), U9.19 (TESTEN), U9.57 (GND), Y2.2, Y2.4
- net LED: now also D6.2 (A), U9.28 (GPIO17)
- net LED_R: now also U10.4 (B)
- net PORT+: now also J3.A6 (D+), J3.B6 (D+), U6.6 (I/O1)
- net PORT-: now also J3.A7 (D-), J3.B7 (D-), U6.4 (I/O2)
- net QSPI_CLK: now also U8.6 (CLK), U9.52 (QSPI_SCLK)
- net QSPI_CS: now also R20.1, R22.2, U8.1 (/CS), U9.56 (QSPI_SS_N)
- net QSPI_SD0: now also U8.5 (DI(IO0)), U9.53 (QSPI_SD0)
- net QSPI_SD1: now also U8.2 (DO(IO1)), U9.55 (QSPI_SD1)
- net QSPI_SD2: now also U8.3 (IO2), U9.54 (QSPI_SD2)
- net QSPI_SD3: now also U8.7 (IO3), U9.51 (QSPI_SD3)
- net RGB_DO: now also U10.3 (A), U9.37 (GPIO25)
- net SCL_L: now also U9.5 (GPIO3)
- net SDA_L: now also U9.4 (GPIO2)
- net SWD_CLK: now also TP3.1, U9.24 (SWCLK)
- net SWD_IO: now also TP4.1, U9.25 (SWDIO)
- net VBUS_DETECT: now also R27.2, R28.1, U9.30 (GPIO19)
- net col0_L: now also U9.12 (GPIO9)
- net col1_L: now also U9.13 (GPIO10)
- net col2_L: now also U9.14 (GPIO11)
- net col3_L: now also U9.15 (GPIO12)
- net col4_L: now also U9.16 (GPIO13)
- net col5_L: now also U9.17 (GPIO14)
- net col6_L: now also U9.18 (GPIO15)
- net data_L: now also U9.2 (GPIO0)
- net row0_L: now also U9.6 (GPIO4)
- net row1_L: now also U9.7 (GPIO5)
- net row2_L: now also U9.8 (GPIO6)
- net row3_L: now also U9.9 (GPIO7)
- net row4_L: now also U9.11 (GPIO8)
- net +5V_R: now reaches J1.1 (A)
- net +5V_R: now also C108.1, D4.1 (K), U10.6 (VCCB), U6.5 (VBUS), U7.3 (EN), U7.4 (Vin)
- new net: Q4.6 (D), R4_L2.1
- new net: C107.1, C6b2.1, Q4.5 (G), R3.1, R4_L2.2
- new net: D6.1 (K), R26.1
- new net: R3.2, R4.1
- new net: C109.2, U9.20 (XTAL_IN), Y2.3
- new net: R25.2, U9.21 (XTAL_OUT)
- new net: D5.1 (K), R21.1
- new net: J3.A5 (CC1), R18.2
- new net: J3.B5 (CC2), R19.2
- new net: FB2.1, J3.S1 (SHIELD)
- new net: C110.2, R25.1, Y2.1
- new net: D4.2 (A), F2.2
- new net: Q3.5 (G), Q3.6 (D), Q4.1 (S), Q4.2 (G), R4b2.2
- new net RESET_R: Q3.2 (G), R3b2.2, SW2.2
- new net RST_R: Q3.3 (D), R3_L2.2, U9.26 (~{RUN})
- new net USB+R: R23.1, U6.1 (I/O1)
- new net USB-R: R24.1, U6.3 (I/O2)
- new net VBUS_R: C6.1, F2.1, J3.A4 (VBUS), J3.A9 (VBUS), J3.B4 (VBUS), J3.B9 (VBUS), R27.1
- no-connect marks 8 -> 12
Other:
- note added: "Reset Circuit Right"
- note added: "USB, ESD protection and Power, Right"
- moved on the sheet: C1, C104, C14, C2, C20, C21, C22, C23, C24, C25, C27, C28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
