File: umiko.kicad_sch (KiCad schematic)
At the start: 414 parts, among them J1 MJ-4PP-9, J2 MJ-4PP-9, J3 USB_C_Receptacle_USB2.0, J5 USB_C_Receptacle_USB2.0, Q1 2N7002VC-, Q2 2N7002VC-, Q3 2N7002VC-, Q4 2N7002VC-, SW1 SWITCH, SW2 SWITCH, U1 USBLC6-2P6, U10 74LVC1T45, U2 TLV75533PDQNR, U3 W25Q128JVPIQ, U4 RP2040, U5 74LVC1T45, U6 USBLC6-2P6, U7 TLV75533PDQNR, U8 W25Q128JVPIQ, U9 RP2040, Y1 12MHz, Y2 12MHz

Commit message: Fix power net separation and clean up old backups
Switch power symbol instances from lib_name to lib_id approach so KiCad 9
correctly resolves separate nets for left/right halves. Remove unwanted
variant lib_symbols and purge old backup zips.

Co-Authored-By: Claude Opus 4.6 <noreply@anthropic.com>
Parts:
- renumbered R22 to R22_R1, R3_L2 to R3_R1, R4_L2 to R4_R1
Connections:
- net GND_R is gone; now on net GND_L: C1.2, C104.2, C107.2, C109.1, C110.1, C111.1, C112.1, C113.2, C114.2, C115.2, C116.2, C117.2, C118.2, C119.2, C120.2, C121.2, C14.2, C2.2, C20.1, C21.2, C22.1, C23.1, C24.2, C25.1, C27.2, C28.1, C3.2, C31.2, C32.2, C33.2, C34.2, C35.2, C36.2, C37.2, C4.2, C48.2, C49.2, C50.2, C51.2, C52.2, C53.2, C54.2, C55.2, C6.2, C65.2, C66.2, C67.2, C68.2, C69.2, C6_A2.2, C6b2.2, C70.2, C71.2, C79.2, C80.2, C81.2, C82.2, C83.2, C84.2, C91.2, C92.2, C93.2, C94.2, C95.2, FB2.2, J1.2 (B), J3.A1 (GND), J3.A12 (GND), J3.B1 (GND), J3.B12 (GND), LED1.3 (VSS), LED104.3 (VSS), LED14.3 (VSS), LED15.3 (VSS), LED16.3 (VSS), LED17.3 (VSS), LED18.3 (VSS), LED19.3 (VSS), LED2.3 (VSS), LED20.3 (VSS), LED22.3 (VSS), LED23.3 (VSS), LED3.3 (VSS), LED31.3 (VSS), LED32.3 (VSS), LED33.3 (VSS), LED34.3 (VSS), LED35.3 (VSS), LED36.3 (VSS), LED4.3 (VSS), LED48.3 (VSS), LED49.3 (VSS), LED50.3 (VSS), LED51.3 (VSS), LED52.3 (VSS), LED53.3 (VSS), LED54.3 (VSS), LED65.3 (VSS), LED66.3 (VSS), LED67.3 (VSS), LED68.3 (VSS), LED69.3 (VSS), LED70.3 (VSS), LED71.3 (VSS), LED79.3 (VSS), LED80.3 (VSS), LED81.3 (VSS), LED82.3 (VSS), LED83.3 (VSS), LED84.3 (VSS), LED91.3 (VSS), LED92.3 (VSS), LED93.3 (VSS), LED94.3 (VSS), Q3.1 (S), Q4.4 (S), R18.1, R19.1, R21.2, R26.2, R28.2, R4.2, SW2.1, U10.2 (GND), U8.4 (GND), U8.9 (GND), U9.19 (TESTEN), U9.57 (GND), Y2.2, Y2.4
- net SCL_L: no longer U9.5 (GPIO3)
- net SDA_L: no longer U9.4 (GPIO2)
- net col0_L: no longer SW_1.1 (COL), SW_18.1 (COL), SW_35.1 (COL), SW_48.1 (COL), SW_61.1 (COL), U9.12 (GPIO9)
- net col1_L: no longer SW_19.1 (COL), SW_2.1 (COL), SW_36.1 (COL), SW_49.1 (COL), U9.13 (GPIO10)
- net col2_L: no longer SW_20.1 (COL), SW_3.1 (COL), SW_37.1 (COL), SW_50.1 (COL), U9.14 (GPIO11)
- net col3_L: no longer SW_21.1 (COL), SW_38.1 (COL), SW_4.1 (COL), SW_51.1 (COL), SW_62.1 (COL), U9.15 (GPIO12)
- net col4_L: no longer SW_22.1 (COL), SW_39.1 (COL), SW_5.1 (COL), SW_52.1 (COL), SW_63.1 (COL), U9.16 (GPIO13)
- net col5_L: no longer SW_23.1 (COL), SW_40.1 (COL), SW_6.1 (COL), U9.17 (GPIO14)
- net col6_L: no longer SW_24.1 (COL), SW_41.1 (COL), SW_53.1 (COL), SW_64.1 (COL), U9.18 (GPIO15)
- net data_L: no longer J1.4 (D), U9.2 (GPIO0)
- net row0_L: no longer D_1.1 (K), D_2.1 (K), D_3.1 (K), D_4.1 (K), D_5.1 (K), D_6.1 (K), D_7.1 (K), U9.6 (GPIO4)
- net row1_L: no longer D_18.1 (K), D_19.1 (K), D_20.1 (K), D_21.1 (K), D_22.1 (K), D_23.1 (K), D_24.1 (K), D_25.1 (K), U9.7 (GPIO5)
- net row2_L: no longer D_35.1 (K), D_36.1 (K), D_37.1 (K), D_38.1 (K), D_39.1 (K), D_40.1 (K), D_41.1 (K), U9.8 (GPIO6)
- net row3_L: no longer D_48.1 (K), D_49.1 (K), D_50.1 (K), D_51.1 (K), D_52.1 (K), D_53.1 (K), U9.9 (GPIO7)
- net row4_L: no longer D_61.1 (K), D_62.1 (K), D_63.1 (K), D_64.1 (K), D_65.1 (K), U9.11 (GPIO8)
- net 16 renamed 16_L
- net 16_L: no longer U9.27 (GPIO16)
- net 1_RX0 renamed 1_RX0_L
- net 1_RX0_L: no longer U9.3 (GPIO1)
- net 20_SDI renamed 20_SDI_L
- net 20_SDI_L: no longer U9.31 (GPIO20)
- net 21_CS renamed 21_CS_L
- net 21_CS_L: no longer U9.32 (GPIO21)
- net 22_SCK renamed 22_SCK_L
- net 22_SCK_L: no longer U9.34 (GPIO22)
- net 23_SDO renamed 23_SDO_L
- net 23_SDO_L: no longer U9.35 (GPIO23)
- net A0 renamed A0_L
- net A0_L: no longer U9.38 (GPIO26/ADC0)
- net A1 renamed A1_L
- net A1_L: no longer U9.39 (GPIO27/ADC1)
- net A2 renamed A2_L
- net A2_L: no longer U9.40 (GPIO28/ADC2)
- net A3 renamed A3_L
- net A3_L: no longer U9.41 (GPIO29/ADC3)
- net BOOT renamed BOOT_L
- net BOOT_L: no longer Q4.3 (D), R20.2
- net D+ renamed D+_L
- net D+_L: no longer R23.2, U9.47 (D+)
- net D- renamed D-_L
- net D-_L: no longer R24.2, U9.46 (D-)
- net LED renamed USER_LED_L
- net USER_LED_L: no longer D6.2 (A), U9.28 (GPIO17)
- net QSPI_CLK renamed QSPI_CLK_L
- net QSPI_CLK_L: no longer U8.6 (CLK), U9.52 (QSPI_SCLK)
- net QSPI_CS renamed QSPI_CS_L
- net QSPI_CS_L: no longer R20.1, R22_R1.2, U8.1 (/CS), U9.56 (QSPI_SS_N)
- net QSPI_SD0 renamed QSPI_SD0_L
- net QSPI_SD0_L: no longer U8.5 (DI(IO0)), U9.53 (QSPI_SD0)
- net QSPI_SD1 renamed QSPI_SD1_L
- net QSPI_SD1_L: no longer U8.2 (DO(IO1)), U9.55 (QSPI_SD1)
- net QSPI_SD2 renamed QSPI_SD2_L
- net QSPI_SD2_L: no longer U8.3 (IO2), U9.54 (QSPI_SD2)
- net QSPI_SD3 renamed QSPI_SD3_L
- net QSPI_SD3_L: no longer U8.7 (IO3), U9.51 (QSPI_SD3)
- net RGB_DO renamed RGB_DO_L
- net RGB_DO_L: no longer U10.3 (A), U9.37 (GPIO25)
- net SWD_CLK renamed SWD_CLK_L
- net SWD_CLK_L: no longer TP3.1, U9.24 (SWCLK)
- net SWD_IO renamed SWD_IO_L
- net SWD_IO_L: no longer TP4.1, U9.25 (SWDIO)
- net VBUS_DETECT renamed VBUS_DETECT_L
- net VBUS_DETECT_L: no longer R27.2, R28.1, U9.30 (GPIO19)
- new net 16_R: U9.27 (GPIO16)
- new net 1_RX0_R: U9.3 (GPIO1)
- new net 20_SDI_R: U9.31 (GPIO20)
- new net 21_CS_R: U9.32 (GPIO21)
- new net 22_SCK_R: U9.34 (GPIO22)
- new net 23_SDO_R: U9.35 (GPIO23)
- new net A0_R: U9.38 (GPIO26/ADC0)
- new net A1_R: U9.39 (GPIO27/ADC1)
- new net A2_R: U9.40 (GPIO28/ADC2)
- new net A3_R: U9.41 (GPIO29/ADC3)
- new net BOOT_R: Q4.3 (D), R20.2
- new net D+_R: R23.2, U9.47 (D+)
- new net D-_R: R24.2, U9.46 (D-)
- new net QSPI_CLK_R: U8.6 (CLK), U9.52 (QSPI_SCLK)
- new net QSPI_CS_R: R20.1, R22_R1.2, U8.1 (/CS), U9.56 (QSPI_SS_N)
- new net QSPI_SD0_R: U8.5 (DI(IO0)), U9.53 (QSPI_SD0)
- new net QSPI_SD1_R: U8.2 (DO(IO1)), U9.55 (QSPI_SD1)
- new net QSPI_SD2_R: U8.3 (IO2), U9.54 (QSPI_SD2)
- new net QSPI_SD3_R: U8.7 (IO3), U9.51 (QSPI_SD3)
- new net RGB_DO_R: U10.3 (A), U9.37 (GPIO25)
- new net SCL_R: U9.5 (GPIO3)
- new net SDA_R: U9.4 (GPIO2)
- new net SWD_CLK_R: TP3.1, U9.24 (SWCLK)
- new net SWD_IO_R: TP4.1, U9.25 (SWDIO)
- new net USER_LED_R: D6.2 (A), U9.28 (GPIO17)
- new net VBUS_DETECT_R: R27.2, R28.1, U9.30 (GPIO19)
- new net col0_R: SW_1.1 (COL), SW_18.1 (COL), SW_35.1 (COL), SW_48.1 (COL), SW_61.1 (COL), U9.12 (GPIO9)
- new net col1_R: SW_19.1 (COL), SW_2.1 (COL), SW_36.1 (COL), SW_49.1 (COL), U9.13 (GPIO10)
- new net col2_R: SW_20.1 (COL), SW_3.1 (COL), SW_37.1 (COL), SW_50.1 (COL), U9.14 (GPIO11)
- new net col3_R: SW_21.1 (COL), SW_38.1 (COL), SW_4.1 (COL), SW_51.1 (COL), SW_62.1 (COL), U9.15 (GPIO12)
- new net col4_R: SW_22.1 (COL), SW_39.1 (COL), SW_5.1 (COL), SW_52.1 (COL), SW_63.1 (COL), U9.16 (GPIO13)
- new net col5_R: SW_23.1 (COL), SW_40.1 (COL), SW_6.1 (COL), U9.17 (GPIO14)
- new net col6_R: SW_24.1 (COL), SW_41.1 (COL), SW_53.1 (COL), SW_64.1 (COL), U9.18 (GPIO15)
- new net data_R: J1.4 (D), U9.2 (GPIO0)
- new net row0_R: D_1.1 (K), D_2.1 (K), D_3.1 (K), D_4.1 (K), D_5.1 (K), D_6.1 (K), D_7.1 (K), U9.6 (GPIO4)
- new net row1_R: D_18.1 (K), D_19.1 (K), D_20.1 (K), D_21.1 (K), D_22.1 (K), D_23.1 (K), D_24.1 (K), D_25.1 (K), U9.7 (GPIO5)
- new net row2_R: D_35.1 (K), D_36.1 (K), D_37.1 (K), D_38.1 (K), D_39.1 (K), D_40.1 (K), D_41.1 (K), U9.8 (GPIO6)
- new net row3_R: D_48.1 (K), D_49.1 (K), D_50.1 (K), D_51.1 (K), D_52.1 (K), D_53.1 (K), U9.9 (GPIO7)
- new net row4_R: D_61.1 (K), D_62.1 (K), D_63.1 (K), D_64.1 (K), D_65.1 (K), U9.11 (GPIO8)
Other:
- moved on the sheet: C1, C10, C100, C101, C102, C103, C104, C107, C108, C109, C11, C110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
