File: umiko.kicad_sch (KiCad schematic)
At the start: 414 parts, among them J1 MJ-4PP-9, J2 MJ-4PP-9, J3 USB_C_Receptacle_USB2.0, J5 USB_C_Receptacle_USB2.0, Q1 2N7002VC-, Q2 2N7002VC-, Q3 2N7002VC-, Q4 2N7002VC-, SW1 SWITCH, SW2 SWITCH, U1 USBLC6-2P6, U10 74LVC1T45, U2 TLV75533PDQNR, U3 W25Q128JVPIQ, U4 RP2040, U5 74LVC1T45, U6 USBLC6-2P6, U7 TLV75533PDQNR, U8 W25Q128JVPIQ, U9 RP2040, Y1 12MHz, Y2 12MHz

Commit message: Place right-side RP2040 passives mirroring left-side layout
Distributed R15-R23, R27, C5b2, C6_A2, C59-C73 around U7
to match the spatial arrangement of left-side passives around U11.

Co-Authored-By: Claude Opus 4.6 <noreply@anthropic.com>
Parts:
- removed C107, C26: 10u, Capacitor_SMD:C_0402_1005Metric, symbol Device:C
- removed C6b1, C6b2: 4.7u, Capacitor_SMD:C_0402_1005Metric, symbol Device:C
- removed Q1, Q2, Q3, Q4: 2N7002VC-, PCM_0xcb:SOT-563, symbol Transistor_FET:FDG6335N
- removed R20, R9: 1k, Resistor_SMD:R_0402_1005Metric, symbol Device:R
- removed R3, R4, R4_L1, R4_R1, R5, R6: 51k, Resistor_SMD:R_0402_1005Metric, symbol Device:R
- removed R3_L1, R3_R1, R3b1, R3b2, R4b1, R4b2: 10k, Resistor_SMD:R_0402_1005Metric, symbol Device:R
- removed U4: RP2040, Package_DFN_QFN:QFN-56-1EP_7x7mm_P0.4mm_EP3.2x3.2mm, symbol 0xcb:RP2040
- added U11: RP2040, Package_DFN_QFN:QFN-56-1EP_7x7mm_P0.4mm_EP3.2x3.2mm, symbol PCM_0xcb:RP2040
- U10: renamed from U7; footprint PCM_0xcb:X2SON-4 -> 0xcb:X2SON-4; symbol 0xcb:LP5907SNX-3.3-NOPB -> PCM_0xcb:LP5907SNX-3.3-NOPB; JLC Basic (none) -> N; LCSC C2861882 -> C133572; Manufacturer (none) -> Texas Instruments; Substitute (none) -> N
- U2: footprint PCM_0xcb:X2SON-4 -> 0xcb:X2SON-4; symbol 0xcb:LP5907SNX-3.3-NOPB -> PCM_0xcb:LP5907SNX-3.3-NOPB; JLC Basic (none) -> N; LCSC C2861882 -> C133572; Manufacturer (none) -> Texas Instruments; Substitute (none) -> N
- U3: footprint PCM_0xcb:W25Q128JVPIQ -> 0xcb:W25Q128JVPIQ; symbol 0xcb:W25Q128JVPIQ -> PCM_0xcb:W25Q128JVPIQ; JLC Basic (none) -> N; Manufacturer (none) -> Winbond; Package (none) -> WSON8-5x6
- U5: value 74LVC1T45 -> SN74LVC1T45DRL; footprint PCM_0xcb:SOT-563 -> Package_TO_SOT_SMD:SOT-563
- U6: renamed from U8; footprint PCM_0xcb:W25Q128JVPIQ -> 0xcb:W25Q128JVPIQ; symbol 0xcb:W25Q128JVPIQ -> PCM_0xcb:W25Q128JVPIQ; JLC Basic (none) -> N; Manufacturer (none) -> Winbond; Package (none) -> WSON8-5x6
- U7: renamed from U9; symbol 0xcb:RP2040 -> PCM_0xcb:RP2040; JLC Basic (none) -> N; Manufacturer (none) -> Raspberry Pi; Package (none) -> LQFN-56_EP_7.0x7.0x0.4P
- U8: renamed from U10; value 74LVC1T45 -> SN74LVC1T45DRL; footprint PCM_0xcb:SOT-563 -> Package_TO_SOT_SMD:SOT-563
- renumbered C41 to C1, C15 to C10, C3 to C100, C23 to C101, C35 to C102, C52 to C103, C69 to C104, C83 to C105, C93 to C106, C4 to C107, C24 to C108, C36 to C109, C43 to C11, C53 to C110, C70 to C111, C25 to C112, C54 to C113, C71 to C114, C84 to C115, C94 to C116, C37 to C117, C55 to C118, C95 to C119, C60 to C12, C27 to C120, C28 to C121, C74 to C13, C86 to C14, C101 to C15, C9 to C16, C16 to C17, C44 to C18, C61 to C19, C59 to C2, C75 to C20, C87 to C21, C102 to C22, C10 to C23, C17 to C24, C45 to C25, C62 to C26, C76 to C27, C88 to C28, C11 to C29, C72 to C3, C18 to C30, C46 to C31, C63 to C32, C77 to C33, C89 to C34, C19 to C35, C12 to C36, C47 to C37, C64 to C38, C78 to C39, C99 to C4, C90 to C40, C103 to C41, C13 to C42, C5 to C43, C29 to C45, C30 to C46, C38 to C47, C39 to C48, C40 to C49, C7 to C5, C56 to C50, C57 to C51, C58 to C52, C85 to C53, C96 to C54, C97 to C55, C98 to C56, C105 to C57, C106 to C58, C109 to C59, C42 to C6, C110 to C60, C111 to C61, C112 to C62, C113 to C63, C114 to C64, C115 to C65, C116 to C66, C117 to C67, C118 to C68, C119 to C69, C73 to C7, C120 to C70, C121 to C71, C6 to C72, C108 to C73, C14 to C75, C31 to C76, C48 to C77, C65 to C78, C100 to C8, C91 to C80, C32 to C81, C49 to C82, C66 to C83, C80 to C84, C1 to C85, C20 to C86, C104 to C87, C21 to C88, C33 to C89, C8 to C9, C50 to C90, C67 to C91, C81 to C92, C34 to C93, C51 to C94, C68 to C95, C82 to C96, C92 to C97, C2 to C98, C22 to C99, D3 to D1, D1 to D2, D2 to D3, D6 to D4, D4 to D5, D5 to D6, D_11 to D_1, D_43 to D_10, D_56 to D_11, D_71 to D_12, D_14 to D_13, D_31 to D_14, D_44 to D_15, D_57 to D_16, D_72 to D_17, D_15 to D_18, D_32 to D_19, D_29 to D_2, D_45 to D_20, D_58 to D_21, D_16 to D_22, D_33 to D_23, D_46 to D_24, D_59 to D_25, D_17 to D_26, D_34 to D_27, D_47 to D_28, D_60 to D_29, D_42 to D_3, D_73 to D_30, D_1 to D_31, D_18 to D_32, D_35 to D_33, D_48 to D_34, D_61 to D_35, D_2 to D_36, D_19 to D_37, D_36 to D_38, D_49 to D_39, D_69 to D_4, D_3 to D_40, D_20 to D_41, D_37 to D_42, D_50 to D_43, D_4 to D_44, D_21 to D_45, D_38 to D_46, D_51 to D_47, D_62 to D_48, D_5 to D_49, D_12 to D_5, D_22 to D_50, D_39 to D_51, D_63 to D_53, D_6 to D_54, D_23 to D_55, D_40 to D_56, D_24 to D_57, D_41 to D_58, D_53 to D_59, D_55 to D_6, D_64 to D_60, D_7 to D_61, D_25 to D_62, D_65 to D_63, D_70 to D_7, D_13 to D_8, D_30 to D_9, J5 to J1, J1 to J3, J3 to J4, LED41 to LED1, LED43 to LED10, LED60 to LED11, LED74 to LED12, LED86 to LED13, LED101 to LED14, LED9 to LED15, LED26 to LED16, LED10 to LED17, LED27 to LED18, LED44 to LED19, LED59 to LED2, LED61 to LED20, LED75 to LED21, LED87 to LED22, LED102 to LED23, LED11 to LED24, LED28 to LED25, LED45 to LED26, LED62 to LED27, LED76 to LED28, LED88 to LED29, LED72 to LED3, LED12 to LED30, LED29 to LED31, LED46 to LED32, LED63 to LED33, LED77 to LED34, LED89 to LED35, LED13 to LED36, LED30 to LED37, LED47 to LED38, LED64 to LED39, LED99 to LED4, LED78 to LED40, LED90 to LED41, LED103 to LED42, LED31 to LED43, LED48 to LED44, LED65 to LED45, LED79 to LED46, LED91 to LED47, LED1 to LED48, LED14 to LED49, LED7 to LED5, LED32 to LED50, LED49 to LED51, LED66 to LED52, LED80 to LED53, LED104 to LED54, LED15 to LED55, LED33 to LED56, LED50 to LED57, LED67 to LED58, LED81 to LED59, LED8 to LED6, LED2 to LED60, LED16 to LED61, LED34 to LED62, LED51 to LED63, LED68 to LED64, LED82 to LED65, LED92 to LED66, LED3 to LED67, LED17 to LED68, LED35 to LED69, LED42 to LED7, LED52 to LED70, LED69 to LED71, LED83 to LED72, LED93 to LED73, LED4 to LED74, LED18 to LED75, LED36 to LED76, LED53 to LED77, LED70 to LED78, LED19 to LED79, LED73 to LED8, LED54 to LED80, LED71 to LED81, LED84 to LED82, LED94 to LED83, LED20 to LED84, LED37 to LED85, LED55 to LED86, LED95 to LED87, LED22 to LED88, LED23 to LED89, LED100 to LED9, R2 to R1, R13 to R10, R14 to R11, R15 to R12, R16 to R13, R17 to R14, R23 to R15, R24 to R16, R25 to R17, R26 to R18, R27 to R19, R28 to R20, R18 to R21, R19 to R22, R21 to R23, R1 to R27, R7 to R4, R8 to R5, R10 to R7, R11 to R8, R12 to R9, SW_11 to SW_1, SW_43 to SW_10, SW_56 to SW_11, SW_71 to SW_12, SW_14 to SW_13, SW_31 to SW_14, SW_44 to SW_15, SW_57 to SW_16, SW_72 to SW_17, SW_15 to SW_18, SW_32 to SW_19, SW_29 to SW_2, SW_45 to SW_20, SW_58 to SW_21, SW_16 to SW_22, SW_33 to SW_23, SW_46 to SW_24, SW_59 to SW_25, SW_17 to SW_26, SW_34 to SW_27, SW_47 to SW_28, SW_60 to SW_29, SW_42 to SW_3, SW_73 to SW_30, SW_1 to SW_31, SW_18 to SW_32, SW_35 to SW_33, SW_48 to SW_34, SW_61 to SW_35, SW_2 to SW_36, SW_19 to SW_37, SW_36 to SW_38, SW_49 to SW_39, SW_69 to SW_4, SW_3 to SW_40, SW_20 to SW_41, SW_37 to SW_42, SW_50 to SW_43, SW_4 to SW_44, SW_21 to SW_45, SW_38 to SW_46, SW_51 to SW_47, SW_62 to SW_48, SW_5 to SW_49, SW_12 to SW_5, SW_22 to SW_50, SW_39 to SW_51, SW_63 to SW_53, SW_6 to SW_54, SW_23 to SW_55, SW_40 to SW_56, SW_24 to SW_57, SW_41 to SW_58, SW_53 to SW_59, SW_55 to SW_6, SW_64 to SW_60, SW_7 to SW_61, SW_25 to SW_62, SW_65 to SW_63, SW_70 to SW_7, SW_13 to SW_8, SW_30 to SW_9, U6 to U9
Connections:
- net RESET_L is gone; now on net QSPI_CS_L: SW1.2
- net RESET_R is gone; now on net QSPI_CS_R: SW2.2
- net +1V1_L: now also U11.23 (DVDD), U11.45 (VREG_VOUT), U11.50 (DVDD); no longer C62.2, C69.1, C71.1, U7.23 (DVDD), U7.45 (VREG_VOUT), U7.50 (DVDD)
- net +3V3_L: now also U11.1 (IOVDD), U11.10 (IOVDD), U11.22 (IOVDD), U11.33 (IOVDD), U11.42 (IOVDD), U11.43 (ADC_AVDD), U11.44 (VREG_VIN), U11.48 (USB_VDD), U11.49 (IOVDD); no longer C5b2.1, C61.2, C63.1, C64.1, C65.1, C66.1, C67.1, C68.1, C6_A2.1, C70.1, D6.2 (A), R22_R1.1, U10.1 (Vout), U6.8 (VCC), U7.1 (IOVDD), U7.10 (IOVDD), U7.22 (IOVDD), U7.33 (IOVDD), U7.42 (IOVDD), U7.43 (ADC_AVDD), U7.44 (VREG_VIN), U7.48 (USB_VDD), U7.49 (IOVDD), U8.1 (VCCA), U8.5 (DIR)
- net 16_L: now also U11.27 (GPIO16)
- net 1_RX0_L: now also U11.3 (GPIO1)
- net 20_SDI_L: now also U11.31 (GPIO20)
- net 21_CS_L: now also U11.32 (GPIO21)
- net 22_SCK_L: now also U11.34 (GPIO22)
- net 23_SDO_L: now also U11.35 (GPIO23)
- net A0_L: now also U11.38 (GPIO26/ADC0)
- net A1_L: now also U11.39 (GPIO27/ADC1)
- net A2_L: now also U11.40 (GPIO28/ADC2)
- net A3_L: now also U11.41 (GPIO29/ADC3)
- net D+_L: now also U11.47 (D+)
- net D-_L: now also U11.46 (D-)
- net GND_L: now also U11.19 (TESTEN), U11.57 (GND); no longer C100.2, C101.1, C102.2, C103.2, C104.2, C105.2, C106.2, C107.2, C108.2, C109.2, C110.2, C111.2, C112.1, C113.2, C114.2, C115.2, C116.2, C117.2, C118.2, C119.2, C120.2, C121.1, C59.1, C5b2.2, C60.1, C61.1, C62.1, C63.2, C64.2, C65.2, C66.2, C67.2, C68.2, C69.2, C6_A2.2, C70.2, C71.2, C72.2, C73.2, C75.2, C76.2, C77.2, C78.2, C79.2, C80.2, C81.2, C82.2, C83.2, C84.2, C85.2, C86.1, C87.2, C88.2, C89.2, C90.2, C91.2, C92.2, C93.2, C94.2, C95.2, C96.2, C97.2, C98.2, C99.1, FB2.2, J3.2 (B), J4.A1 (GND), J4.A12 (GND), J4.B1 (GND), J4.B12 (GND), LED43.3 (VSS), LED44.3 (VSS), LED45.3 (VSS), LED46.3 (VSS), LED47.3 (VSS), LED48.3 (VSS), LED49.3 (VSS), LED50.3 (VSS), LED51.3 (VSS), LED52.3 (VSS), LED53.3 (VSS), LED54.3 (VSS), LED55.3 (VSS), LED56.3 (VSS), LED57.3 (VSS), LED58.3 (VSS), LED59.3 (VSS), LED60.3 (VSS), LED61.3 (VSS), LED62.3 (VSS), LED63.3 (VSS), LED64.3 (VSS), LED65.3 (VSS), LED66.3 (VSS), LED67.3 (VSS), LED68.3 (VSS), LED69.3 (VSS), LED70.3 (VSS), LED71.3 (VSS), LED72.3 (VSS), LED73.3 (VSS), LED74.3 (VSS), LED75.3 (VSS), LED76.3 (VSS), LED77.3 (VSS), LED78.3 (VSS), LED79.3 (VSS), LED80.3 (VSS), LED81.3 (VSS), LED82.3 (VSS), LED83.3 (VSS), LED84.3 (VSS), LED88.3 (VSS), LED89.3 (VSS), R18.2, R20.2, R21.1, R22.1, R23.2, R4.1, R5.1, SW2.1, U10.2 (GND), U10.5 (TP), U6.4 (GND), U6.9 (GND), U7.19 (TESTEN), U7.57 (GND), U8.2 (GND), U9.2 (GND), Y2.2, Y2.4
- net QSPI_CLK_L: now also U11.52 (QSPI_SCLK)
- net QSPI_CS_L: now also U11.56 (QSPI_SS_N)
- net QSPI_SD0_L: now also U11.53 (QSPI_SD0)
- net QSPI_SD1_L: now also U11.55 (QSPI_SD1)
- net QSPI_SD2_L: now also U11.54 (QSPI_SD2)
- net QSPI_SD3_L: now also U11.51 (QSPI_SD3)
- net RGB_DO_L: now also U11.37 (GPIO25)
- net SCL_L: now also U11.5 (GPIO3)
- net SDA_L: now also U11.4 (GPIO2)
- net SWD_CLK_L: now also U11.24 (SWCLK)
- net SWD_IO_L: now also U11.25 (SWDIO)
- net USER_LED_L: now also U11.28 (GPIO17)
- net VBUS_DETECT_L: now also U11.30 (GPIO19)
- net col0_L: now also U11.12 (GPIO9)
- net col1_L: now also U11.13 (GPIO10)
- net col2_L: now also U11.14 (GPIO11)
- net col3_L: now also U11.15 (GPIO12)
- net col4_L: now also U11.16 (GPIO13)
- net col5_L: now also U11.17 (GPIO14)
- net col6_L: now also U11.18 (GPIO15)
- net data_L: now also U11.2 (GPIO0)
- net row0_L: now also U11.6 (GPIO4)
- net row1_L: now also U11.7 (GPIO5)
- net row2_L: now also U11.8 (GPIO6)
- net row3_L: now also U11.9 (GPIO7)
- net row4_L: now also U11.11 (GPIO8)
- net GND_R: now reaches LED85.3 (VSS), LED86.3 (VSS), LED87.3 (VSS)
- net GND_R: now also C100.2, C101.1, C102.2, C103.2, C104.2, C105.2, C106.2, C107.2, C108.2, C109.2, C110.2, C111.2, C112.1, C113.2, C114.2, C115.2, C116.2, C117.2, C118.2, C119.2, C120.2, C121.1, C59.1, C5b2.2, C60.1, C61.1, C62.1, C63.2, C64.2, C65.2, C66.2, C67.2, C68.2, C69.2, C6_A2.2, C70.2, C71.2, C72.2, C73.2, C75.2, C76.2, C77.2, C78.2, C79.2, C80.2, C81.2, C82.2, C83.2, C84.2, C85.2, C86.1, C87.2, C88.2, C89.2, C90.2, C91.2, C92.2, C93.2, C94.2, C95.2, C96.2, C97.2, C98.2, C99.1, FB2.2, J3.2 (B), J4.A1 (GND), J4.A12 (GND), J4.B1 (GND), J4.B12 (GND), LED43.3 (VSS), LED44.3 (VSS), LED45.3 (VSS), LED46.3 (VSS), LED47.3 (VSS), LED48.3 (VSS), LED49.3 (VSS), LED50.3 (VSS), LED51.3 (VSS), LED52.3 (VSS), LED53.3 (VSS), LED54.3 (VSS), LED55.3 (VSS), LED56.3 (VSS), LED57.3 (VSS), LED58.3 (VSS), LED59.3 (VSS), LED60.3 (VSS), LED61.3 (VSS), LED62.3 (VSS), LED63.3 (VSS), LED64.3 (VSS), LED65.3 (VSS), LED66.3 (VSS), LED67.3 (VSS), LED68.3 (VSS), LED69.3 (VSS), LED70.3 (VSS), LED71.3 (VSS), LED72.3 (VSS), LED73.3 (VSS), LED74.3 (VSS), LED75.3 (VSS), LED76.3 (VSS), LED77.3 (VSS), LED78.3 (VSS), LED79.3 (VSS), LED80.3 (VSS), LED81.3 (VSS), LED82.3 (VSS), LED83.3 (VSS), LED84.3 (VSS), LED88.3 (VSS), LED89.3 (VSS), R18.2, R20.2, R21.1, R22.1, R23.2, SW2.1, U10.2 (GND), U10.5 (TP), U6.4 (GND), U6.9 (GND), U7.19 (TESTEN), U7.57 (GND), U8.2 (GND), U9.2 (GND), Y2.2, Y2.4; no longer LED74.2 (DOUT)
- net at LED87.4 (DIN): now also LED74.2 (DOUT)
- net at C46.2, Y1.3: now also U11.20 (XTAL_IN)
- net at R11.2: now also U11.21 (XTAL_OUT)
- net PORT+ renamed PORT_L+
- net PORT_L+: no longer J4.A6 (D+), J4.B6 (D+), U9.6 (I/O1)
- net PORT- renamed PORT_L-
- net PORT_L-: no longer J4.A7 (D-), J4.B7 (D-), U9.4 (I/O2)
- new net: R4.1, R5.1
- new net +1V1_R: C62.2, C69.1, C71.1, U7.23 (DVDD), U7.45 (VREG_VOUT), U7.50 (DVDD)
- new net +3V3_R: C5b2.1, C61.2, C63.1, C64.1, C65.1, C66.1, C67.1, C68.1, C6_A2.1, C70.1, D6.2 (A), R22_R1.1, U10.1 (Vout), U6.8 (VCC), U7.1 (IOVDD), U7.10 (IOVDD), U7.22 (IOVDD), U7.33 (IOVDD), U7.42 (IOVDD), U7.43 (ADC_AVDD), U7.44 (VREG_VIN), U7.48 (USB_VDD), U7.49 (IOVDD), U8.1 (VCCA), U8.5 (DIR)
- new net PORT_R+: J4.A6 (D+), J4.B6 (D+), U9.6 (I/O1)
- new net PORT_R-: J4.A7 (D-), J4.B7 (D-), U9.4 (I/O2)
- no-connect marks 12 -> 32
Other:
- note removed: "Delay Circuit"
- note removed: "Reset Circuit Left"
- note removed: "Reset Circuit Right"
- moved on the sheet: C100, C101, C102, C103, C104, C105, C106, C107, C108, C109, C110, C111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

Commit message: Add SWD debug TP5-TP8 and arrange pads for pogo-clip access
Added four test points (TP5/TP6 for GND_L/+3V3_L, TP7/TP8 for
GND_R/+3V3_R) in the schematic and PCB, and repositioned all 8
SWD-related test pads into mirrored vertical columns at 2.54mm
pitch with 1.27mm pads, sized for an Adafruit 6-pin pogo clip.
Left column reads CLK/IO/GND/3V3 top-to-bottom; right column
mirrors as 3V3/GND/IO/CLK so a flipped clip lands on matching
signals on both halves. Added F.SilkS function labels and hid
the TPn references on silkscreen.

Co-Authored-By: Claude Opus 4.7 (1M context) <noreply@anthropic.com>
Parts:
- added TP5, TP7: GND, PCM_0xcb:TestPoint_Pad_D0.8mm, symbol Connector:TestPoint_Small
- added TP6, TP8: 3V3, PCM_0xcb:TestPoint_Pad_D0.8mm, symbol Connector:TestPoint_Small
Connections:
- net +3V3_L: now also TP6.1
- net +3V3_R: now also TP8.1
- net GND_L: now also R4.1, R5.1, TP5.1
- net GND_R: now also TP7.1

Commit message: Tighten net classes and add inner GND pours
- Default netclass: track 0.1->0.2mm, via 0.46/0.2 -> 0.6/0.3
- New GND netclass at 0.3mm; GND_L/GND_R routed through it instead of Default
- Normalize GND_L/GND_R, VBUS_L/R, +5V_L/R, USB +/- track widths to class spec
  (preserve intentional wider segments)
- Add In2.Cu GND_L and GND_R copper pours mirroring B.Cu outlines so the
  inner layer is a continuous ground floor
- Snap dangling Edge.Cuts endpoints (right-half top edge had a 23um vertical
  mismatch); both halves now form closed loops at 5um tolerance

Co-Authored-By: Claude Opus 4.7 (1M context) <noreply@anthropic.com>
Connections:
- net RST_R: no longer names the net of U7.26 (~{RUN})

Commit message: Soften corners, clean library refs, drop OLED remnants
- Edge.Cuts corners enlarged to 2mm fillets, then fully unfilleted to
  sharp 90deg in preparation for board squish (both halves still form
  closed loops at 5um tolerance).
- Schematic Footprint property fixed for U2/U3/U6/U10: '0xcb:' prefix
  corrected to 'PCM_0xcb:' so Update PCB from Schematic resolves.
- Removed two orphan Display:ER_OLEDM0.91_1x-I2C footprints (REF**, no
  schematic counterpart) leftover from the dropped OLED design.

Co-Authored-By: Claude Opus 4.7 (1M context) <noreply@anthropic.com>
Parts:
- removed J2, J3: MJ-4PP-9, mj-4pp-9:MJ-4PP-9, symbol mj-4pp-9:MJ-4PP-9
- added J3, J4: USB_C_Receptacle_USB2.0, PCM_0xcb:USB_C_Receptacle_HRO_TYPE-C-31-M-12, symbol Connector:USB_C_Receptacle_USB2.0
- U10, U2: footprint 0xcb:X2SON-4 -> PCM_0xcb:X2SON-4
- U3, U6: footprint 0xcb:W25Q128JVPIQ -> PCM_0xcb:W25Q128JVPIQ
- renumbered J4 to J2
Connections:
- net +5V_L: now also J3.A4 (VBUS), J3.A9 (VBUS), J3.B4 (VBUS), J3.B9 (VBUS)
- net +5V_R: now also J4.A4 (VBUS), J4.A9 (VBUS), J4.B4 (VBUS), J4.B9 (VBUS)
- net GND_L: now also J3.A1 (GND), J3.A12 (GND), J3.B1 (GND), J3.B12 (GND)
- net GND_R: now also J4.A1 (GND), J4.A12 (GND), J4.B1 (GND), J4.B12 (GND)
- net data_L: now also J3.A6 (D+), J3.B6 (D+)
- net data_R: now also J4.A6 (D+), J4.B6 (D+)
- no-connect marks 32 -> 30

Commit message: Major PCB cleanup: inner USB-C planks, 3D models, TP alignment
- Add J3/J4 inner USB-C planks at 10mm from inner edges, mirror-symmetric.
- Normalize all Edge.Cuts to canonical y values; both halves still
  closed loops.
- Fix library prefix on U2/U3/U6/U10 (0xcb -> PCM_0xcb) so
  Update PCB from Schematic resolves.
- Remove orphan OLED footprints leftover from dropped OLED design.
- Mirror right-side TPs to match left-side Y range, fix x positions
  to 2.5mm from actual inner edges (was 0.58mm after edge moved).
- Shrink F.Fab/B.Fab text to 0.25mm; tune silk to 0.5mm.
- Remap all 3D model paths to current install (KICAD10_3DMODEL_DIR);
  fix WRL->STEP for v10 install; substitute LED_0402 for D_0402;
  map Mac hardcoded path to local onigaku.
- Add Gateron KS-33 v2.0 switch body 3D model to all 63 switches
  (z=-4.1 offset, 180-Z rotation for B.Cu auto-flip handling).
- Fix underglow LED footprints: header layer F.Cu -> B.Cu so KiCad
  renders them below the board; adjust model rotation accordingly.
- README: note Kailh Choc V2 stabilizer cutouts, add KS-33 3D model
  TODO.

Co-Authored-By: Claude Opus 4.7 (1M context) <noreply@anthropic.com>
Parts:
- removed D_17: D, onigaku:D3_SMD_v2, symbol Device:D_Small
- removed SW_17: KEYSW, Gateron_KS33_Hotswap:Gateron-KS33-Hotswap-1.25U, symbol MX_Alps_Hybrid:MX-NoLED
Changed lines of the file:
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@@
 	)
 	(junction
-		(at 124.46 175.26)
-		(diameter 0)
-		(color 0 0 0 0)
-	)
-	(junction
 		(at 109.22 234.95)
 		(diameter 0)
@@
 	)
 	(junction
-		(at 135.89 138.43)
-		(diameter 1.016)
-		(color 0 0 0 0)
-	)
-	(junction
 		(at 277.114 132.334)
 		(diameter 0)
@@
 	(wire
 		(pts
-			(xy 124.46 168.91) (xy 124.46 170.18)
-		)
-		(stroke
-			(width 0)
-			(type solid)
-		)
-	)
-	(wire
-		(pts
 			(xy 270.51 71.12) (xy 270.51 72.39)
 		)
@@
 	(wire
 		(pts
-			(xy 124.46 175.26) (xy 200.66 175.26)
-		)
-		(stroke
-			(width 0)
-			(type solid)
-		)
-	)
-	(wire
-		(pts
 			(xy 439.42 131.318) (xy 444.5 131.318)
 		)
@@
 	(wire
 		(pts
-			(xy 99.06 175.26) (xy 124.46 175.26)
+			(xy 99.06 175.26) (xy 200.66 175.26)
 		)
 		(stroke
@@
 	(wire
 		(pts
-			(xy 129.54 163.83) (xy 135.89 163.83)
-		)
-		(stroke
-			(width 0)
-			(type solid)
-		)
-	)
-	(wire
-		(pts
 			(xy 129.54 62.23) (xy 135.89 62.23)
 		)
@@
 	(wire
 		(pts
-			(xy 135.89 163.83) (xy 135.89 138.43)
-		)
-		(stroke
-			(width 0)
-			(type solid)
-		)
-	)
-	(wire
-		(pts
 			(xy 607.568 70.358) (xy 607.568 71.628)
 		)
@@
 	)
 	(symbol
-		(lib_id "Device:D_Small")
-		(at 124.46 172.72 90)
-		(unit 1)
-		(body_style 1)
-		(exclude_from_sim no)
-		(in_bom yes)
-		(on_board yes)
-		(in_pos_files yes)
-		(dnp no)
-		(property "Reference" "D_17"
-			(at 127 170.942 90)
-			(show_name no)
-			(do_not_autoplace no)
-			(effects
-				(font
-					(size 1.27 1.27)
-				)
-				(justify right)
-			)
-		)
-		(property "Value" "D"
-			(at 127 173.228 90)
-			(show_name no)
-			(do_not_autoplace no)
-			(effects
-				(font
-					(size 1.27 1.27)
-				)
-				(justify right)
-			)
-		)
-		(property "Footprint" "onigaku:D3_SMD_v2"
-			(at 124.46 172.72 90)
-			(hide yes)
-			(show_name no)
-			(do_not_autoplace no)
-			(effects
-				(font
-					(size 1.27 1.27)
-				)
-			)
-		)
-		(property "Datasheet" ""
-			(at 124.46 172.72 90)
-			(hide yes)
-			(show_name no)
-			(do_not_autoplace no)
-			(effects
-				(font
-					(size 1.27 1.27)
-				)
-			)
-		)
-		(property "Description" "Diode, small symbol"
-			(at 124.46 172.72 0)
-			(hide yes)
-			(show_name no)
-			(do_not_autoplace no)
-			(effects
-				(font
-					(size 1.27 1.27)
-				)
-			)
-		)
-		(property "Sim.Device" "D"
-			(at 124.46 172.72 0)
-			(hide yes)
-			(show_name no)
-			(do_not_autoplace no)
-			(effects
-				(font
-					(size 1.27 1.27)
-				)
-			)
-		)
-		(property "Sim.Pins" "1=K 2=A"
-			(at 124.46 172.72 0)
-			(hide yes)
-			(show_name no)
-			(do_not_autoplace no)
-			(effects
-				(font
-					(size 1.27 1.27)
-				)
-			)
-		)
-		(pin "2"
-		)
-		(pin "1"
-		)
-		(instances
-			(project "umiko"
-				(path "/4b4aa2f9-db35-4fc9-9772-4a4fa5dd4e1a"
-					(reference "D_17")
-					(unit 1)
-				)
-			)
-		)
-	)
-	(symbol
 		(lib_id "Device:C_Small")
 		(at 152.4 285.75 0)
@@
 					(unit 1)
 				)
-			)
-		)
-	)
-	(symbol
-		(lib_id "MX_Alps_Hybrid:MX-NoLED")
-		(at 125.73 165.1 0)
-		(unit 1)
-		(body_style 1)
-		(exclude_from_sim no)
-		(in_bom yes)
-		(on_board yes)
-		(in_pos_files yes)
-		(dnp no)
-		(property "Reference" "SW_17"
-			(at 125.73 159.1818 0)
-			(show_name no)
-			(do_not_autoplace no)
-			(effects
-				(font
-					(size 1.524 1.524)
-				)
-			)
-		)
-		(property "Value" "KEYSW"
-			(at 125.73 167.64 0)
-			(hide yes)
-			(show_name no)
-			(do_not_autoplace no)
-			(effects
-				(font
-					(size 1.524 1.524)
-				)
-			)
-		)
-		(property "Footprint" "Gateron_KS33_Hotswap:Gateron-KS33-Hotswap-1.25U"
-			(at 125.73 165.1 0)
-			(hide yes)
-			(show_name no)
-			(do_not_autoplace no)
-			(effects
-				(font
-					(size 1.524 1.524)
-				)
-			)
-		)
-		(property "Datasheet" ""
-			(at 125.73 165.1 0)
-			(show_name no)
-			(do_not_autoplace no)
-			(effects
-				(font
-					(size 1.524 1.524)
-				)
-			)
-		)
-		(property "Description" ""
-			(at 125.73 165.1 0)
-			(show_name no)
-			(do_not_autoplace no)
-			(effects
-				(font
-					(size 1.27 1.27)
-				)
-			)
-		)
-		(pin "1"
-		)
-		(pin "2"
-		)
-		(instances
-			(project "umiko"
-				(path "/4b4aa2f9-db35-4fc9-9772-4a4fa5dd4e1a"
-					(reference "SW_17")
-					(unit 1)
-				)

Commit message: Add JLC/CAD export scripts, restore SW_17/D_17, refresh BOM
- make_jlc_files.py: kicad-cli wrapper that emits JLC-ready gerbers/BOM/CPL
  with the strict formatting JLC's parser actually wants (integer rotations,
  4-decimal coords, mm suffix, fullwidth parens in BOM header, aux-origin
  alignment across all three outputs). LCSC overrides for D3_SMD_v2 and
  SK6812MINI-E so JLC auto-matches them on upload.
- make_cad_files.py: per-component-group STEP exports plus per-half STEPs
  for SolidWorks case design (avoids the flat multibody dump).
- Restore SW_17 / D_17 to schematic and link C22, D_17, LED23 footprints
  back to their schematic UUIDs in the PCB.
- README: BOM table now carries LCSC part numbers; new sections covering
  the JLC re-upload gotcha and the CPL format quirks discovered during fab.
- Rename umiko-* artwork footprints to bakekujira-* to track the upstream
  library rename; refresh splash/back-graphic image assets.
- Prune old umiko-backups; keep recent snapshots.

Co-Authored-By: Claude Opus 4.7 (1M context) <noreply@anthropic.com>
Parts:
- added D_17: D, onigaku:D3_SMD_v2, symbol Device:D_Small
- added SW_17: KEYSW, Gateron_KS33_Hotswap:Gateron-KS33-Hotswap-1.25U, symbol MX_Alps_Hybrid:MX-NoLED
Connections:
- net col3_L: now also SW_17.1 (COL)
- net row4_L: now also D_17.1 (K)
- new net: D_17.2 (A), SW_17.2 (ROW)
Changed lines of the file:
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@@
 	)
 	(junction
+		(at 124.46 175.26)
+		(diameter 0)
+		(color 0 0 0 0)
+	)
+	(junction
 		(at 109.22 234.95)
 		(diameter 0)
@@
 	)
 	(junction
+		(at 135.89 138.43)
+		(diameter 1.016)
+		(color 0 0 0 0)
+	)
+	(junction
 		(at 277.114 132.334)
 		(diameter 0)
@@
 	(wire
 		(pts
+			(xy 124.46 168.91) (xy 124.46 170.18)
+		)
+		(stroke
+			(width 0)
+			(type solid)
+		)
+	)
+	(wire
+		(pts
 			(xy 270.51 71.12) (xy 270.51 72.39)
 		)
@@
 	(wire
 		(pts
+			(xy 124.46 175.26) (xy 200.66 175.26)
+		)
+		(stroke
+			(width 0)
+			(type solid)
+		)
+	)
+	(wire
+		(pts
 			(xy 439.42 131.318) (xy 444.5 131.318)
 		)
@@
 	(wire
 		(pts
-			(xy 99.06 175.26) (xy 200.66 175.26)
+			(xy 99.06 175.26) (xy 124.46 175.26)
 		)
 		(stroke
@@
 	(wire
 		(pts
+			(xy 129.54 163.83) (xy 135.89 163.83)
+		)
+		(stroke
+			(width 0)
+			(type solid)
+		)
+	)
+	(wire
+		(pts
 			(xy 129.54 62.23) (xy 135.89 62.23)
 		)
@@
 	(wire
 		(pts
+			(xy 135.89 163.83) (xy 135.89 138.43)
+		)
+		(stroke
+			(width 0)
+			(type solid)
+		)
+	)
+	(wire
+		(pts
 			(xy 607.568 70.358) (xy 607.568 71.628)
 		)
@@
 	)
 	(symbol
+		(lib_id "Device:D_Small")
+		(at 124.46 172.72 90)
+		(unit 1)
+		(body_style 1)
+		(exclude_from_sim no)
+		(in_bom yes)
+		(on_board yes)
+		(in_pos_files yes)
+		(dnp no)
+		(property "Reference" "D_17"
+			(at 127 170.942 90)
+			(show_name no)
+			(do_not_autoplace no)
+			(effects
+				(font
+					(size 1.27 1.27)
+				)
+				(justify right)
+			)
+		)
+		(property "Value" "D"
+			(at 127 173.228 90)
+			(show_name no)
+			(do_not_autoplace no)
+			(effects
+				(font
+					(size 1.27 1.27)
+				)
+				(justify right)
+			)
+		)
+		(property "Footprint" "onigaku:D3_SMD_v2"
+			(at 124.46 172.72 90)
+			(hide yes)
+			(show_name no)
+			(do_not_autoplace no)
+			(effects
+				(font
+					(size 1.27 1.27)
+				)
+			)
+		)
+		(property "Datasheet" ""
+			(at 124.46 172.72 90)
+			(hide yes)
+			(show_name no)
+			(do_not_autoplace no)
+			(effects
+				(font
+					(size 1.27 1.27)
+				)
+			)
+		)
+		(property "Description" "Diode, small symbol"
+			(at 124.46 172.72 0)
+			(hide yes)
+			(show_name no)
+			(do_not_autoplace no)
+			(effects
+				(font
+					(size 1.27 1.27)
+				)
+			)
+		)
+		(property "Sim.Device" "D"
+			(at 124.46 172.72 0)
+			(hide yes)
+			(show_name no)
+			(do_not_autoplace no)
+			(effects
+				(font
+					(size 1.27 1.27)
+				)
+			)
+		)
+		(property "Sim.Pins" "1=K 2=A"
+			(at 124.46 172.72 0)
+			(hide yes)
+			(show_name no)
+			(do_not_autoplace no)
+			(effects
+				(font
+					(size 1.27 1.27)
+				)
+			)
+		)
+		(pin "2"
+		)
+		(pin "1"
+		)
+		(instances
+			(project "umiko"
+				(path "/4b4aa2f9-db35-4fc9-9772-4a4fa5dd4e1a"
+					(reference "D_17")
+					(unit 1)
+				)
+			)
+		)
+	)
+	(symbol
 		(lib_id "Device:C_Small")
 		(at 152.4 285.75 0)
@@
 					(unit 1)
 				)
+			)
+		)
+	)
+	(symbol
+		(lib_id "MX_Alps_Hybrid:MX-NoLED")
+		(at 125.73 165.1 0)
+		(unit 1)
+		(body_style 1)
+		(exclude_from_sim no)
+		(in_bom yes)
+		(on_board yes)
+		(in_pos_files yes)
+		(dnp no)
+		(property "Reference" "SW_17"
+			(at 125.73 159.1818 0)
+			(show_name no)
+			(do_not_autoplace no)
+			(effects
+				(font
+					(size 1.524 1.524)
+				)
+			)
+		)
+		(property "Value" "KEYSW"
+			(at 125.73 167.64 0)
+			(hide yes)
+			(show_name no)
+			(do_not_autoplace no)
+			(effects
+				(font
+					(size 1.524 1.524)
+				)
+			)
+		)
+		(property "Footprint" "Gateron_KS33_Hotswap:Gateron-KS33-Hotswap-1.25U"
+			(at 125.73 165.1 0)
+			(hide yes)
+			(show_name no)
+			(do_not_autoplace no)
+			(effects
+				(font
+					(size 1.524 1.524)
+				)
+			)
+		)
+		(property "Datasheet" ""
+			(at 125.73 165.1 0)
+			(show_name no)
+			(do_not_autoplace no)
+			(effects
+				(font
+					(size 1.524 1.524)
+				)
+			)
+		)
+		(property "Description" ""
+			(at 125.73 165.1 0)
+			(show_name no)
+			(do_not_autoplace no)
+			(effects
+				(font
+					(size 1.27 1.27)
+				)
+			)
+		)
+		(pin "1"
+		)
+		(pin "2"
+		)
+		(instances
+			(project "umiko"
+				(path "/4b4aa2f9-db35-4fc9-9772-4a4fa5dd4e1a"
+					(reference "SW_17")
+					(unit 1)
+				)

Commit message: Swap inter-half USB-C for TRRS; resize polyfuse; side-mount host USB-C
Major reorganization of the split-keyboard connectors:

- Replaced inter-half USB-C (J3/J4) with TRRS (U4/U12, keebio:TRRS symbol
  + onigaku:TRRS-PJ-320A footprint on B.Cu). RP2040 PIO serial only needs
  GND + Data + 5V; TRRS RING2 reserved spare. Existing D1/D5 Schottkys
  already provide diode-OR on the 5V bridge — no extra parts needed.
- Bumped polyfuses F1/F2 from 500mA to 1.1A (Bourns MF-PSMF110X-2, LCSC
  C89658, same 0603 footprint) for RGB headroom across the split bridge.
- Moved host USB-Cs J1/J2 to the outer side edges of each half.
- Replaced 7mm-tall inner USB-C planks (P2/P3) with 2mm flush-to-inner-
  edge TRRS planks (8mm wide, 0.5mm fillets on outer + inner-top corners).
- Replaced 7mm-tall outer USB-C planks (P1/P4) with 2mm side planks on
  the outer edges to support the new J1/J2 placement; 3mm protrusion
  leaves ~1mm of body overhang for cable clearance.
- Re-enabled keebio fp library; added 3D model reference for the TRRS
  jacks (PJ320A.step from onigaku/packages3D).

Includes one-shot patch scripts for the plank surgery (kept for
reference): plank flush, 1mm shift, notch removal, corner bevel, side
planks, and the 1.5mm shrink.

Co-Authored-By: Claude Opus 4.7 (1M context) <noreply@anthropic.com>
Parts:
- removed J3, J4: USB_C_Receptacle_USB2.0, PCM_0xcb:USB_C_Receptacle_HRO_TYPE-C-31-M-12, symbol Connector:USB_C_Receptacle_USB2.0
- added U12, U4: TRRS, onigaku:TRRS-PJ-320A, symbol keebio:TRRS
- F1, F2: value 500mA -> 1.1A; LCSC C210357 -> C89658; MPN MF-FSMF050X-2 -> MF-PSMF110X-2
Connections:
- net +5V_L: now also U4.2 (TIP)
- net +5V_R: now also U12.2 (TIP)
- net GND_L: now also U4.1 (SLEEVE)
- net GND_R: now also U12.1 (SLEEVE)
- net data_L: now also U4.3 (RING1)
- net data_R: now also U12.3 (RING1)
- no-connect marks 30 -> 33
