File: umiko.kicad_sch (KiCad schematic)
At the start: 396 parts, among them J1 USB_C_Receptacle_USB2.0, J2 USB_C_Receptacle_USB2.0, J3 USB_C_Receptacle_USB2.0, J4 USB_C_Receptacle_USB2.0, SW1 SWITCH, SW2 SWITCH, U1 USBLC6-2P6, U10 TLV75533PDQNR, U11 RP2040, U2 TLV75533PDQNR, U3 W25Q128JVPIQ, U5 SN74LVC1T45DRL, U6 W25Q128JVPIQ, U7 RP2040, U8 SN74LVC1T45DRL, U9 USBLC6-2P6, Y1 12MHz, Y2 12MHz

Commit message: Manual schematic + PCB updates from KiCad GUI
Hand work after the top-mount J3/J4 migration: re-routing inter-half USB-C
nets, layout cleanup, and other in-KiCad refinements.

Co-Authored-By: Claude Opus 4.7 <noreply@anthropic.com>
Parts:
- added C122: 0.1uF, Capacitor_SMD:C_0603_1608Metric_Pad1.08x0.95mm_HandSolder, symbol Device:C_Small
- added LED90: YS-SK6812MINI-E, onigaku:YS-SK6812MINI-E_underglow, symbol umiko-rescue:YS-SK6812MINI-E-kbd
Connections:
- net +5V_R: now also C122.2, LED90.1 (VDD)
- net GND_R: now also C122.1, LED90.3 (VSS)
- net at LED55.4 (DIN): now also LED90.2 (DOUT); no longer LED61.2 (DOUT)
- new net: LED61.2 (DOUT), LED90.4 (DIN)

Commit message: USB-C shield: expose S2/S3/S4 in symbol + J2 area routing pass
Schematic: added S2/S3/S4 SHIELD pins to the embedded
Connector:USB_C_Receptacle_USB2.0 symbol so all four shield/mounting pads
can be wired (previously only S1 was exposed). PCB: routing pass on the
right host USB-C (J2) area.

Co-Authored-By: Claude Opus 4.7 <noreply@anthropic.com>
Connections:
- net GND_L: now also J1.S2 (SHIELD), J1.S3 (SHIELD), J1.S4 (SHIELD), J3.S1 (SHIELD), J3.S2 (SHIELD), J3.S3 (SHIELD), J3.S4 (SHIELD)
- net GND_R: now also J2.S2 (SHIELD), J2.S3 (SHIELD), J2.S4 (SHIELD), J4.S1 (SHIELD), J4.S2 (SHIELD), J4.S3 (SHIELD), J4.S4 (SHIELD)

Commit message: Refactor plate generator to read-only + start OLED placement
- scripts/_gen_plate_cutouts.py -> scripts/make_plate.py: read-only on
  source PCB. All transforms (inject cutouts, build STEP-ready board)
  happen in memory; a single self-deleting temp PCB is what kicad-cli
  reads. The source umiko.kicad_pcb is never modified by the script.
- README: reference make_plate.py and note both make_* scripts are
  read-only on the source PCB.
- PCB/schematic: in-progress OLED footprint + I2C wiring + related
  refinements from the KiCad session.

Co-Authored-By: Claude Opus 4.7 <noreply@anthropic.com>
Parts:
- added R24, R25, R26, R6: 5.1k, Resistor_SMD:R_0402_1005Metric, symbol Device:R
- added R28, R29, R30, R31: 4.7k, Resistor_SMD:R_0402_1005Metric, symbol Device:R
- added U12, U4: SSD1306, onigaku:OLED_v2, symbol PCM_0xcb:SSD1306
Connections:
- net +3V3_L: now also R28.1, R29.1, U4.2 (VCC)
- net +3V3_R: now also R30.1, R31.1, U12.2 (VCC)
- net GND_L: now also R24.1, R6.1, U4.1 (GND)
- net GND_R: now also R25.1, R26.1, U12.1 (GND)
- net SCL_L: now also R28.2, U4.3 (SCL)
- net SCL_R: now also R30.2, U12.3 (SCL)
- net SDA_L: now also R29.2, U4.4 (SDA)
- net SDA_R: now also R31.2, U12.4 (SDA)
- net at J3.A5 (CC1): now also R6.2
- net at J3.B5 (CC2): now also R24.2
- net at J4.A5 (CC1): now also R25.2
- net at J4.B5 (CC2): now also R26.2

Commit message: OLED placement work-in-progress
In-KiCad placement and footprint work for the right-half OLED + initial
sizing exploration for the left-half display location.

Co-Authored-By: Claude Opus 4.7 <noreply@anthropic.com>
Parts:
- removed R28, R29: 4.7k, Resistor_SMD:R_0402_1005Metric, symbol Device:R
- removed U4: SSD1306, onigaku:OLED_v2, symbol PCM_0xcb:SSD1306

Commit message: Fix wrong LCSC code on USB-C connectors J1-J4
C963373 (G-Switch GT-USB-7014C, pure-SMD mid-mount) was a mismatch for
our HRO TYPE-C-31-M-12 footprint (SMD signals + THT shield legs + NPTH
alignment pegs). JLC flagged it during engineering review of order
SMT026060360534. Correct LCSC for HRO TYPE-C-31-M-12 is C165948.

Also clarify line 111 of README: drop misleading "mid-mount-ish"
description in favor of the actual mounting topology.

Co-Authored-By: Claude Opus 4.7 <noreply@anthropic.com>
Parts:
- J1, J2, J3, J4: LCSC C963373 -> C165948
Changed lines of the file:
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@@
 			)
 		)
-		(property "LCSC" "C963373"
+		(property "LCSC" "C165948"
 			(at 439.928 204.724 0)
 			(hide yes)
@@
 			)
 		)
-		(property "LCSC" "C963373"
+		(property "LCSC" "C165948"
 			(at 403.098 74.168 0)
 			(hide yes)
@@
 			)
 		)
-		(property "LCSC" "C963373"
+		(property "LCSC" "C165948"
 			(at 512.064 188.214 0)
 			(hide yes)
@@
 			)
 		)
-		(property "LCSC" "C963373"
+		(property "LCSC" "C165948"
 			(at 255.27 73.66 0)
 			(hide yes)

Commit message: Fix F1/F2 polyfuse part mismatch: C89658 (0805) -> C210357 (0603)
The 0603 fuse footprint we copied from the 0xCB Helios reference design
was paired with the wrong LCSC code (C89658 = Bourns MF-PSMF110X-2, which
is 0805 / 1.1 A). JLC flagged the body-vs-pad mismatch on order
SMT026060360534 (Phoebe's second review).

Helios actually uses C210357 = Bourns MF-FSMF050X-2, a real 0603 part
rated 500 mA hold / 1 A trip. Swap to that. 500 mA is comfortable
headroom for a keyboard (typical draw <300 mA with all LEDs lit) and
trips on real fault current, so it's still protective.

Value field updated 1.1A -> 500mA to keep BOM rows accurate.

Co-Authored-By: Claude Opus 4.7 <noreply@anthropic.com>
Parts:
- F1, F2: value 1.1A -> 500mA; LCSC C89658 -> C210357
Changed lines of the file:
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@@
 			)
 		)
-		(property "Value" "1.1A"
+		(property "Value" "500mA"
 			(at 429.768 61.468 90)
 			(show_name no)
@@
 			)
 		)
-		(property "LCSC" "C89658"
+		(property "LCSC" "C210357"
 			(at 429.768 58.928 0)
 			(hide yes)
@@
 			)
 		)
-		(property "Value" "1.1A"
+		(property "Value" "500mA"
 			(at 281.94 60.96 90)
 			(show_name no)
@@
 			)
 		)
-		(property "LCSC" "C89658"
+		(property "LCSC" "C210357"
 			(at 281.94 58.42 0)
 			(hide yes)

Commit message: Fix LDO label drift: U2/U10 honestly say LP5907SNX-3.3
Backstory: U2/U10 schematic Value and MPN fields said TLV75533PDQNR
(Helios reference design) but the actual placed chip has been LP5907SNX-3.3
since JLC ran out of TLV75533 in the X2SON-4 package. The two are
pin-compatible drop-ins for the same footprint, but the BOM saying one
thing while the board has another was misleading for anyone reading the
repo without the conversation context.

Sync Value, MPN, LCSC, Footprint, Datasheet on U2/U10 to consistently
describe the LP5907 that's actually placed. No PCB geometry change; no
schematic-symbol change; no re-routing. LCSC C133572 (LP5907SNX-3.3)
is already correct in the schematic — only the human-readable labels
were drifting.

Considered swapping to TLV75533PDBVR (SOT-23-5, C404027) to match
Helios's 500 mA design intent, but per-half 3.3 V draw on umiko is
~150 mA peak (per-key RGB runs from VBUS 5 V, not the 3.3 V rail), so
the LP5907's 250 mA gives 1.7x headroom over actual load. Swapping
would have meant a new PCB rev for zero operational benefit. Documented
the trade-off in README's new "LDO history" section so future-me can
re-evaluate if v2 adds 3.3 V load.

Co-Authored-By: Claude Opus 4.7 <noreply@anthropic.com>
Parts:
- U10, U2: value TLV75533PDQNR -> LP5907SNX-3.3; MPN TLV75533PDQNR -> LP5907SNX-3.3
Changed lines of the file:
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@@
 			)
 		)
-		(property "Value" "TLV75533PDQNR"
+		(property "Value" "LP5907SNX-3.3"
 			(at 475.488 67.818 0)
 			(show_name no)
@@
 			)
 		)
-		(property "MPN" "TLV75533PDQNR"
+		(property "MPN" "LP5907SNX-3.3"
 			(at 475.488 61.468 0)
 			(hide yes)
@@
 			)
 		)
-		(property "Value" "TLV75533PDQNR"
+		(property "Value" "LP5907SNX-3.3"
 			(at 327.66 67.31 0)
 			(show_name no)
@@
 			)
 		)
-		(property "MPN" "TLV75533PDQNR"
+		(property "MPN" "LP5907SNX-3.3"
 			(at 327.66 60.96 0)
 			(hide yes)

Commit message: Add QMK firmware scaffold + fix col7_R schematic omission
Firmware:
- keyboards/umiko/ scaffolded in fresh QMK clone at ~/dev/keyboard/qmk_umiko
- Copy in firmware/keyboards/umiko/ for source control (keyboard.json,
  rules.mk, config.h, keymaps/default/keymap.c, readme.md)
- 5x8 scanning matrix (rows GP4-GP8, cols GP9-GP16), split serial vendor
  driver on GP0 (single-wire PIO on D+ of J3/J4), COL2ROW, 63-key
  LAYOUT_all with physical positions extracted from the schematic
- Default keymap: QWERTY-ish TKL F-row-less baseline + placeholder Fn layer

Verified compile: umiko_default.uf2 (~74 KB) builds cleanly under
MSYS2 MINGW64 + arm-none-eabi-gcc + qmk 1.2.0.

Hardware (col7_R fix):
- Right MCU U7 GPIO16 wired to col7_R in schematic and PCB, restoring
  SW_61/62/63 (far-right pinky column: Delete, Tab, Control per keymap).
  Original schematic had col7_R as a dangling global label that never
  connected to U7 — SW_61/62/63 were unreachable on the fab-run boards.
  Firmware is built for the fixed 5x8 matrix; on current boards, those 3
  positions register as KC_NO (silent). Post-respin, all 63 keys work
  with the same firmware. No respin ordered yet — validating with
  bridged L+R test first.

README:
- Rewrote QMK toolchain section with the exact recipe that worked
  (MSYS2 packages, jsonschema pinning to avoid rpds-py Rust build,
  USERPROFILE requirement, keyboard.json vs info.json, junction to
  make QMK's default qmk_firmware path resolve to our clone).
- Added scripts/qmk_compile.sh wrapper so future compiles don't
  need to remember the MSYS2 env-var dance.

Co-Authored-By: Claude Opus 4.7 <noreply@anthropic.com>
Parts:
- U12: footprint onigaku:OLED_v2 -> onigaku:OLED_SSD1306_32x12mm
Connections:
- net 16_R is gone; now on net col7_R: U7.27 (GPIO16)
- net 16_L: no longer names the net of U11.27 (GPIO16)
- no-connect marks 31 -> 30
